File: boards/driver/current_drivers.sch (KiCad schematic (older format))
At the start: 121 parts, among them Q1 NMOS, Q10 NMOS, Q11 NMOS, Q12 NMOS, Q13 NMOS, Q14 NMOS, Q15 NMOS, Q16 NMOS, Q17 NMOS, Q18 NMOS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

Commit message: Driver board: added strand selection and return circuits
Changed lines of the file:
@@
 $Descr USLedger 17000 11000
 encoding utf-8
-Sheet 3 3
+Sheet 4 4
 Title ""
 Date ""
@@
 	7500 8600 7600 8500
 Text HLabel 4750 1450 0    50   Input ~ 0
-~IL0[1..8]
+~IL[01..08]
 Wire Bus Line
 	4800 1450 4750 1450
 Text HLabel 4750 1350 0    50   Input ~ 0
-IL0[1..8]
+IL[01..08]
 Wire Bus Line
 	4950 1350 4750 1350
@@
 Connection ~ 13700 1650
 Text HLabel 13900 1550 2    50   Output ~ 0
-XFN0[1..8]
+XFN[01..08]
 Text HLabel 13900 1650 2    50   Output ~ 0
-XCN0[1..8]
+XCN[01..08]
 Wire Bus Line
 	3750 1750 3750 3150
