File: boards/driver/fpga_power.sch (KiCad schematic (older format))
At the start: 40 parts, among them J1 Barrel_Jack_Switch, J2 Conn_01x24, J3 Conn_02x06_Top_Bottom, J4 Conn_01x24, Q90 IRF7413, U10 74LVC245, U11 74LVC245, U12 JTE0624D05, U13 LTC4231-1, U14 74HC4514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

Commit message: Added LED footprints and ignored bitstream files
Parts:
- D160, D161, D162: footprint (none) -> LED_SMD:LED_0603_1608Metric
- R270, R271: footprint (none) -> Resistor_SMD:R_0603_1608Metric
Changed lines of the file:
@@
 F 0 "R270" V 5545 1800 50  0000 C CNN
 F 1 "12k" V 5636 1800 50  0000 C CNN
-F 2 "" V 5790 1790 50  0001 C CNN
+F 2 "Resistor_SMD:R_0603_1608Metric" V 5790 1790 50  0001 C CNN
 F 3 "~" H 5750 1800 50  0001 C CNN
 	1    5750 1800
@@
 F 0 "R271" V 5545 2250 50  0000 C CNN
 F 1 "2.4k" V 5636 2250 50  0000 C CNN
-F 2 "" V 5790 2240 50  0001 C CNN
+F 2 "Resistor_SMD:R_0603_1608Metric" V 5790 2240 50  0001 C CNN
 F 3 "~" H 5750 2250 50  0001 C CNN
 	1    5750 2250
@@
 F 0 "D162" V 9089 1932 50  0000 R CNN
 F 1 "ORANGE" V 8998 1932 50  0000 R CNN
-F 2 "" H 9050 2050 50  0001 C CNN
+F 2 "LED_SMD:LED_0603_1608Metric" H 9050 2050 50  0001 C CNN
 F 3 "~" H 9050 2050 50  0001 C CNN
 	1    9050 2050
@@
 F 0 "D161" V 5339 3132 50  0000 R CNN
 F 1 "TEAL" V 5248 3132 50  0000 R CNN
-F 2 "" H 5300 3250 50  0001 C CNN
+F 2 "LED_SMD:LED_0603_1608Metric" H 5300 3250 50  0001 C CNN
 F 3 "~" H 5300 3250 50  0001 C CNN
 	1    5300 3250
@@
 F 0 "D160" V 4750 3100 50  0000 R CNN
 F 1 "BLUE" V 4850 3100 50  0000 R CNN
-F 2 "" H 4800 3250 50  0001 C CNN
+F 2 "LED_SMD:LED_0603_1608Metric" H 4800 3250 50  0001 C CNN
 F 3 "~" H 4800 3250 50  0001 C CNN
 	1    4800 3250

Commit message: Driver board: largely fleshed out part selection
Parts:
- C50: Digikey (none) -> https://www.digikey.com/en/products/detail/samsung-electro-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; Part Number (none) -> CL10B103KC8NNNC; Rating (none) -> 100V; Tolerance (none) -> 10%
- D160: Digikey (none) -> https://www.digikey.com/en/products/detail/rohm-semiconduct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; Part Number (none) -> SMLD12BN1WT86
- D161: Digikey (none) -> https://www.digikey.com/en/products/detail/rohm-semiconduct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; Part Number (none) -> SMLD12E3N1WT86
- D162: Digikey (none) -> https://www.digikey.com/en/products/detail/stanley-electric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; Part Number (none) -> SJW1151CKS-100-TR
- J1: footprint Connector_BarrelJack:BarrelJack_Horizontal -> lachesis:BarrelJack_CUI_PJ-002A; Digikey (none) -> https://www.digikey.com/en/products/detail/PJ-002A/CP-002A-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; Part Number (none) -> PJ-002A
- Q90: Digikey (none) -> https://www.digikey.com/en/products/detail/infineon-technol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; Part Number (none) -> IRF7413
- U10, U11: Digikey (none) -> https://www.digikey.com/en/products/detail/SN74LVC245APWRG4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; Part Number (none) -> SN74LVC245APWRG4
- U13: Digikey (none) -> https://www.digikey.com/en/products/detail/LTC4231CMS-1%23P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; Part Number (none) -> LTC4231-1
- U14: Digikey (none) -> https://www.digikey.com/en/products/detail/CD74HC4514M96/29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; Part Number (none) -> CD74HC4514M96
- U15, U16, U17, U18: Digikey (none) -> https://www.digikey.com/en/products/detail/SN74LVC2G04DBVT/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; Part Number (none) -> SN74LVC2G04DBVT
Changed lines of the file:
@@
 F 2 "Package_SO:TSSOP-20_4.4x6.5mm_P0.65mm" H 3450 5650 50  0001 C CNN
 F 3 "http://www.ti.com/lit/gpn/sn74HC245" H 3450 5650 50  0001 C CNN
+F 4 "https://www.digikey.com/en/products/detail/SN74LVC245APWRG4/296-31913-1-ND/3506158" H 3450 5650 50  0001 C CNN "Digikey"
+F 5 "SN74LVC245APWRG4" H 3450 5650 50  0001 C CNN "Part Number"
 	1    3450 5650
 	1    0    0    -1
@@
 F 2 "Package_SO:TSSOP-20_4.4x6.5mm_P0.65mm" H 3450 7950 50  0001 C CNN
 F 3 "http://www.ti.com/lit/gpn/sn74HC245" H 3450 7950 50  0001 C CNN
+F 4 "https://www.digikey.com/en/products/detail/SN74LVC245APWRG4/296-31913-1-ND/3506158" H 3450 7950 50  0001 C CNN "Digikey"
+F 5 "SN74LVC245APWRG4" H 3450 7950 50  0001 C CNN "Part Number"
 	1    3450 7950
 	1    0    0    -1
@@
 F 2 "Package_TO_SOT_SMD:SOT-23-6" H 13400 2900 50  0001 C CNN
 F 3 "http://www.ti.com/lit/sg/scyt129e/scyt129e.pdf" H 13400 2900 50  0001 C CNN
+F 4 "https://www.digikey.com/en/products/detail/SN74LVC2G04DBVT/296-26612-1-ND/2255070" H 13400 2900 50  0001 C CNN "Digikey"
+F 5 "SN74LVC2G04DBVT" H 13400 2900 50  0001 C CNN "Part Number"
 	1    13400 2900
 	1    0    0    -1
@@
 F 2 "Package_TO_SOT_SMD:SOT-23-6" H 13400 3200 50  0001 C CNN
 F 3 "http://www.ti.com/lit/sg/scyt129e/scyt129e.pdf" H 13400 3200 50  0001 C CNN
+F 4 "https://www.digikey.com/en/products/detail/SN74LVC2G04DBVT/296-26612-1-ND/2255070" H 13400 3200 50  0001 C CNN "Digikey"
+F 5 "SN74LVC2G04DBVT" H 13400 3200 50  0001 C CNN "Part Number"
 	2    13400 3200
 	1    0    0    -1
@@
 F 2 "Package_TO_SOT_SMD:SOT-23-6" H 13400 3500 50  0001 C CNN
 F 3 "http://www.ti.com/lit/sg/scyt129e/scyt129e.pdf" H 13400 3500 50  0001 C CNN
+F 4 "https://www.digikey.com/en/products/detail/SN74LVC2G04DBVT/296-26612-1-ND/2255070" H 13400 3500 50  0001 C CNN "Digikey"
+F 5 "SN74LVC2G04DBVT" H 13400 3500 50  0001 C CNN "Part Number"
 	1    13400 3500
 	1    0    0    -1
@@
 F 2 "Package_TO_SOT_SMD:SOT-23-6" H 13400 3800 50  0001 C CNN
 F 3 "http://www.ti.com/lit/sg/scyt129e/scyt129e.pdf" H 13400 3800 50  0001 C CNN
+F 4 "https://www.digikey.com/en/products/detail/SN74LVC2G04DBVT/296-26612-1-ND/2255070" H 13400 3800 50  0001 C CNN "Digikey"
+F 5 "SN74LVC2G04DBVT" H 13400 3800 50  0001 C CNN "Part Number"
 	2    13400 3800
 	1    0    0    -1
@@
 F 2 "Package_TO_SOT_SMD:SOT-23-6" H 13400 4100 50  0001 C CNN
 F 3 "http://www.ti.com/lit/sg/scyt129e/scyt129e.pdf" H 13400 4100 50  0001 C CNN
+F 4 "https://www.digikey.com/en/products/detail/SN74LVC2G04DBVT/296-26612-1-ND/2255070" H 13400 4100 50  0001 C CNN "Digikey"
+F 5 "SN74LVC2G04DBVT" H 13400 4100 50  0001 C CNN "Part Number"
 	1    13400 4100
 	1    0    0    -1
@@
 F 2 "Package_TO_SOT_SMD:SOT-23-6" H 13400 4400 50  0001 C CNN
 F 3 "http://www.ti.com/lit/sg/scyt129e/scyt129e.pdf" H 13400 4400 50  0001 C CNN
+F 4 "https://www.digikey.com/en/products/detail/SN74LVC2G04DBVT/296-26612-1-ND/2255070" H 13400 4400 50  0001 C CNN "Digikey"
+F 5 "SN74LVC2G04DBVT" H 13400 4400 50  0001 C CNN "Part Number"
 	2    13400 4400
 	1    0    0    -1
@@
 F 2 "Package_TO_SOT_SMD:SOT-23-6" H 13400 4700 50  0001 C CNN
 F 3 "http://www.ti.com/lit/sg/scyt129e/scyt129e.pdf" H 13400 4700 50  0001 C CNN
+F 4 "https://www.digikey.com/en/products/detail/SN74LVC2G04DBVT/296-26612-1-ND/2255070" H 13400 4700 50  0001 C CNN "Digikey"
+F 5 "SN74LVC2G04DBVT" H 13400 4700 50  0001 C CNN "Part Number"
 	1    13400 4700
 	1    0    0    -1
@@
 F 2 "Package_TO_SOT_SMD:SOT-23-6" H 13400 5000 50  0001 C CNN
 F 3 "http://www.ti.com/lit/sg/scyt129e/scyt129e.pdf" H 13400 5000 50  0001 C CNN
+F 4 "https://www.digikey.com/en/products/detail/SN74LVC2G04DBVT/296-26612-1-ND/2255070" H 13400 5000 50  0001 C CNN "Digikey"
+F 5 "SN74LVC2G04DBVT" H 13400 5000 50  0001 C CNN "Part Number"
 	2    13400 5000
 	1    0    0    -1
@@
 F 2 "Package_TO_SOT_SMD:SOT-23-6" H 13950 7900 50  0001 C CNN
 F 3 "http://www.ti.com/lit/sg/scyt129e/scyt129e.pdf" H 13950 7900 50  0001 C CNN
+F 4 "https://www.digikey.com/en/products/detail/SN74LVC2G04DBVT/296-26612-1-ND/2255070" H 13950 7900 50  0001 C CNN "Digikey"
+F 5 "SN74LVC2G04DBVT" H 13950 7900 50  0001 C CNN "Part Number"
 	3    13950 7900
 	1    0    0    -1
@@
 F 2 "Package_TO_SOT_SMD:SOT-23-6" H 14550 7900 50  0001 C CNN
 F 3 "http://www.ti.com/lit/sg/scyt129e/scyt129e.pdf" H 14550 7900 50  0001 C CNN
+F 4 "https://www.digikey.com/en/products/detail/SN74LVC2G04DBVT/296-26612-1-ND/2255070" H 14550 7900 50  0001 C CNN "Digikey"
+F 5 "SN74LVC2G04DBVT" H 14550 7900 50  0001 C CNN "Part Number"
 	3    14550 7900
 	1    0    0    -1
@@
 F 2 "Package_TO_SOT_SMD:SOT-23-6" H 15150 7900 50  0001 C CNN
 F 3 "http://www.ti.com/lit/sg/scyt129e/scyt129e.pdf" H 15150 7900 50  0001 C CNN
+F 4 "https://www.digikey.com/en/products/detail/SN74LVC2G04DBVT/296-26612-1-ND/2255070" H 15150 7900 50  0001 C CNN "Digikey"
+F 5 "SN74LVC2G04DBVT" H 15150 7900 50  0001 C CNN "Part Number"
 	3    15150 7900
 	1    0    0    -1
@@
 F 2 "Package_SO:SOIC-24W_7.5x15.4mm_P1.27mm" H 10250 7750 50  0001 C CNN
 F 3 "" H 10250 7750 50  0001 C CNN
+F 4 "https://www.digikey.com/en/products/detail/CD74HC4514M96/296-29484-1-ND/2747415" H 10250 7750 50  0001 C CNN "Digikey"
+F 5 "CD74HC4514M96" H 10250 7750 50  0001 C CNN "Part Number"
 	1    10250 7750
 	1    0    0    -1
@@
 F 2 "Package_TO_SOT_SMD:SOT-23-6" H 13350 7900 50  0001 C CNN
 F 3 "http://www.ti.com/lit/sg/scyt129e/scyt129e.pdf" H 13350 7900 50  0001 C CNN
+F 4 "https://www.digikey.com/en/products/detail/SN74LVC2G04DBVT/296-26612-1-ND/2255070" H 13350 7900 50  0001 C CNN "Digikey"
+F 5 "SN74LVC2G04DBVT" H 13350 7900 50  0001 C CNN "Part Number"
 	3    13350 7900
 	1    0    0    -1
@@
 F 2 "Package_SO:MSOP-12_3x4mm_P0.65mm" H 7250 2900 50  0001 C CNN
 F 3 "" H 7250 2900 50  0001 C CNN
+F 4 "https://www.digikey.com/en/products/detail/LTC4231CMS-1%23PBF/LTC4231CMS-1%23PBF-ND/4964746" H 7400 3200 50  0001 C CNN "Digikey"
+F 5 "LTC4231-1" H 7400 3200 50  0001 C CNN "Part Number"
 	1    7400 3200
 	1    0    0    -1
@@
 F 2 "Capacitor_SMD:C_0603_1608Metric" H 8138 2300 50  0001 C CNN
 F 3 "~" H 8100 2450 50  0001 C CNN
+F 4 "https://www.digikey.com/en/products/detail/samsung-electro-mechanics/CL10B103KC8NNNC/3886854" H 8100 2450 50  0001 C CNN "Digikey"
+F 5 "CL10B103KC8NNNC" H 8100 2450 50  0001 C CNN "Part Number"
+F 6 "100V" H 8100 2450 50  0001 C CNN "Rating"
+F 7 "10%" H 8100 2450 50  0001 C CNN "Tolerance"
 	1    8100 2450
 	1    0    0    -1
@@
 F 0 "J1" H 2457 1867 50  0000 C CNN
 F 1 "Barrel_Jack_Switch" H 2457 1776 50  0000 C CNN
-F 2 "Connector_BarrelJack:BarrelJack_Horizontal" H 2450 1510 50  0001 C CNN
+F 2 "lachesis:BarrelJack_CUI_PJ-002A" H 2450 1510 50  0001 C CNN
 F 3 "~" H 2450 1510 50  0001 C CNN
+F 4 "https://www.digikey.com/en/products/detail/PJ-002A/CP-002A-ND/96962" H 2400 1550 50  0001 C CNN "Digikey"
+F 5 "PJ-002A" H 2400 1550 50  0001 C CNN "Part Number"
 	1    2400 1550
 	1    0    0    -1
@@
 F 2 "Package_SO:SO-8_3.9x4.9mm_P1.27mm" H 7750 1650 50  0001 C CNN
 F 3 "~" H 7550 1550 50  0001 C CNN
+F 4 "https://www.digikey.com/en/products/detail/infineon-technologies/IRF7413ZTRPBF/812705" H 7550 1550 50  0001 C CNN "Digikey"
+F 5 "IRF7413" H 7550 1550 50  0001 C CNN "Part Number"
 	1    7550 1550
 	0    -1   -1   0
@@
 F 2 "LED_SMD:LED_0603_1608Metric" H 9050 2050 50  0001 C CNN
 F 3 "~" H 9050 2050 50  0001 C CNN
+F 4 "https://www.digikey.com/en/products/detail/stanley-electric-co/SJW1151CKS-100-TR/8544257?s=N4IgjCBcpgbFoDGUBmBDANgZwKYBoQB7KAbRAGYBOAJgBZ4BdAgBwBcoQBlVgJwEsAdgHMQAXwIBWahIQhkkdNnxFSFABzVyE2iCYg2Hbv2FiCAWmqz5vAK7LikMjIajXQA" H 9050 2050 50  0001 C CNN "Digikey"
+F 5 "SJW1151CKS-100-TR" H 9050 2050 50  0001 C CNN "Part Number"
 	1    9050 2050
 	0    -1   -1   0
@@
 F 2 "LED_SMD:LED_0603_1608Metric" H 5300 3250 50  0001 C CNN
 F 3 "~" H 5300 3250 50  0001 C CNN
+F 4 "https://www.digikey.com/en/products/detail/rohm-semiconductor/SMLD12E3N1WT86/9826161?s=N4IgjCBcpgbFoDGUBmBDANgZwKYBoQB7KAbRAGYBOAJgBZ4BdAgBwBcoQBlVgJwEsAdgHMQAXwLkA7AhDJI6bPiKkK1AAyww0piDYdu-YWIKxKMuQtwFikMrTWUq5EDr2QuvQSPEgAtNXMoXgBXJRsyAFYXURigA" H 5300 3250 50  0001 C CNN "Digikey"
+F 5 "SMLD12E3N1WT86" H 5300 3250 50  0001 C CNN "Part Number"
 	1    5300 3250
 	0    -1   -1   0
@@
 F 2 "LED_SMD:LED_0603_1608Metric" H 4800 3250 50  0001 C CNN
 F 3 "~" H 4800 3250 50  0001 C CNN
+F 4 "https://www.digikey.com/en/products/detail/rohm-semiconductor/SMLD12BN1WT86/9826162?s=N4IgTCBcDaIMoFkAyARAjGAQgOTQdRAF0BfIA" H 4800 3250 50  0001 C CNN "Digikey"
+F 5 "SMLD12BN1WT86" H 4800 3250 50  0001 C CNN "Part Number"
 	1    4800 3250
 	0    -1   1    0
