File: boards/driver/parity.sch (KiCad schematic (older format))
At the start: 11 parts, among them Q86 MMBT2222, Q87 MMBT2222

Commit message: Driver board: largely fleshed out part selection
Parts:
- D152, D153, D154, D155: Digikey (none) -> https://www.digikey.com/en/products/detail/smc-diode-soluti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; Part Number (none) -> 1N4148WSTR
- L37: DCR (none) -> 0.7; Digikey (none) -> https://www.digikey.com/en/products/detail/api-delevan-inc/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; Part Number (none) -> 1812R-222J; Rating (none) -> 535mA; Tolerance (none) -> 5%
- Q86, Q87: Digikey (none) -> https://www.digikey.com/en/products/detail/MMBT2222A-G/641-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; Part Number (none) -> MMBT2222A-G
Changed lines of the file:
@@
 F 2 "Package_TO_SOT_SMD:SOT-23" H 5100 3800 50  0001 C CNN
 F 3 "~" H 4900 3700 50  0001 C CNN
+F 4 "https://www.digikey.com/en/products/detail/MMBT2222A-G/641-1942-1-ND/9477875" H 4900 3700 50  0001 C CNN "Digikey"
+F 5 "MMBT2222A-G" H 4900 3700 50  0001 C CNN "Part Number"
 	1    4900 3700
 	1    0    0    -1
@@
 F 2 "Diode_SMD:D_SOD-323" V 5600 4300 50  0001 C CNN
 F 3 "~" V 5600 4300 50  0001 C CNN
+F 4 "1N4148WSTR" V 4900 3150 50  0001 C CNN "Part Number"
+F 5 "https://www.digikey.com/en/products/detail/smc-diode-solutions/1N4148WSTR/6022449" V 4900 3150 50  0001 C CNN "Digikey"
 	1    5600 4300
 	0    -1   -1   0
@@
 F 2 "Diode_SMD:D_SOD-323" V 5600 4050 50  0001 C CNN
 F 3 "~" V 5600 4050 50  0001 C CNN
+F 4 "1N4148WSTR" V 4900 3150 50  0001 C CNN "Part Number"
+F 5 "https://www.digikey.com/en/products/detail/smc-diode-solutions/1N4148WSTR/6022449" V 4900 3150 50  0001 C CNN "Digikey"
 	1    5600 4050
 	0    -1   -1   0
@@
 F 2 "Diode_SMD:D_SOD-323" V 5600 3800 50  0001 C CNN
 F 3 "~" V 5600 3800 50  0001 C CNN
+F 4 "1N4148WSTR" V 4900 3150 50  0001 C CNN "Part Number"
+F 5 "https://www.digikey.com/en/products/detail/smc-diode-solutions/1N4148WSTR/6022449" V 4900 3150 50  0001 C CNN "Digikey"
 	1    5600 3800
 	0    -1   -1   0
@@
 F 2 "Package_TO_SOT_SMD:SOT-23" H 6250 3450 50  0001 C CNN
 F 3 "~" H 6050 3350 50  0001 C CNN
+F 4 "https://www.digikey.com/en/products/detail/MMBT2222A-G/641-1942-1-ND/9477875" H 6050 3350 50  0001 C CNN "Digikey"
+F 5 "MMBT2222A-G" H 6050 3350 50  0001 C CNN "Part Number"
 	1    6050 3350
 	1    0    0    -1
@@
 F 2 "Diode_SMD:D_SOD-323" V 6150 4800 50  0001 C CNN
 F 3 "~" V 6150 4800 50  0001 C CNN
+F 4 "1N4148WSTR" V 4900 3150 50  0001 C CNN "Part Number"
+F 5 "https://www.digikey.com/en/products/detail/smc-diode-solutions/1N4148WSTR/6022449" V 4900 3150 50  0001 C CNN "Digikey"
 	1    6150 4800
 	0    -1   -1   0
@@
 F 2 "Inductor_SMD:L_1812_4532Metric" H 6150 4450 50  0001 C CNN
 F 3 "~" H 6150 4450 50  0001 C CNN
+F 4 "0.7" H 6150 4450 50  0001 C CNN "DCR"
+F 5 "https://www.digikey.com/en/products/detail/api-delevan-inc/1812R-222J/1115305" H 6150 4450 50  0001 C CNN "Digikey"
+F 6 "1812R-222J" H 6150 4450 50  0001 C CNN "Part Number"
+F 7 "535mA" H 6150 4450 50  0001 C CNN "Rating"
+F 8 "5%" H 6150 4450 50  0001 C CNN "Tolerance"
 	1    6150 4450
 	1    0    0    -1
