File: boards/driver/return.sch (KiCad schematic (older format))
At the start: 14 parts

Commit message: Driver board: a bit more schematic work and some initial footprint selections
Parts:
- R222, R223, R224: footprint Resistor_SMD:R_1206_3216Metric -> Resistor_SMD:R_0603_1608Metric
Changed lines of the file:
@@
 F 0 "R225" V 5005 4850 50  0000 C CNN
 F 1 "200" V 4914 4850 50  0000 C CNN
-F 2 "Resistor_SMD:R_1206_3216Metric" V 4840 4840 50  0001 C CNN
+F 2 "Resistor_SMD:R_0603_1608Metric" V 4840 4840 50  0001 C CNN
 F 3 "~" H 4800 4850 50  0001 C CNN
 	1    4800 4850
@@
 F 0 "R226" V 5955 4850 50  0000 C CNN
 F 1 "200" V 5864 4850 50  0000 C CNN
-F 2 "Resistor_SMD:R_1206_3216Metric" V 5790 4840 50  0001 C CNN
+F 2 "Resistor_SMD:R_0603_1608Metric" V 5790 4840 50  0001 C CNN
 F 3 "~" H 5750 4850 50  0001 C CNN
 	1    5750 4850
@@
 F 0 "R227" V 6905 4850 50  0000 C CNN
 F 1 "200" V 6814 4850 50  0000 C CNN
-F 2 "Resistor_SMD:R_1206_3216Metric" V 6740 4840 50  0001 C CNN
+F 2 "Resistor_SMD:R_0603_1608Metric" V 6740 4840 50  0001 C CNN
 F 3 "~" H 6700 4850 50  0001 C CNN
 	1    6700 4850

Commit message: Driver board: significant cleanup. Moved sense amp pairs into a subsheet, split tuning resistors into two globally, pushed input circuits into their corresponding sheets.
Parts:
- renumbered R222 to R251, R223 to R252, R224 to R253
Changed lines of the file:
@@
 $Descr A4 11693 8268
 encoding utf-8
-Sheet 60 69
+Sheet 60 64
 Title ""
 Date ""
@@
 	5100 5000 5050 5000
 $Comp
-L Device:R_US R222
+L Device:R_US R251
 U 1 1 625E8581
 P 4800 4850
-AR Path="/6183FAE6/625CAD37/625E8581" Ref="R222"  Part="1"
-AR Path="/6183FAE6/6261206B/625E8581" Ref="R225"  Part="1"
-F 0 "R225" V 5005 4850 50  0000 C CNN
+AR Path="/6183FAE6/625CAD37/625E8581" Ref="R251"  Part="1"
+AR Path="/6183FAE6/6261206B/625E8581" Ref="R254"  Part="1"
+F 0 "R254" V 5005 4850 50  0000 C CNN
 F 1 "200" V 4914 4850 50  0000 C CNN
 F 2 "Resistor_SMD:R_0603_1608Metric" V 4840 4840 50  0001 C CNN
@@
 	6050 5000 6000 5000
 $Comp
-L Device:R_US R223
+L Device:R_US R252
 U 1 1 625F4D0E
 P 5750 4850
-AR Path="/6183FAE6/625CAD37/625F4D0E" Ref="R223"  Part="1"
-AR Path="/6183FAE6/6261206B/625F4D0E" Ref="R226"  Part="1"
-F 0 "R226" V 5955 4850 50  0000 C CNN
+AR Path="/6183FAE6/625CAD37/625F4D0E" Ref="R252"  Part="1"
+AR Path="/6183FAE6/6261206B/625F4D0E" Ref="R255"  Part="1"
+F 0 "R255" V 5955 4850 50  0000 C CNN
 F 1 "200" V 5864 4850 50  0000 C CNN
 F 2 "Resistor_SMD:R_0603_1608Metric" V 5790 4840 50  0001 C CNN
@@
 	7000 5000 6950 5000
 $Comp
-L Device:R_US R224
+L Device:R_US R253
 U 1 1 625F8C2E
 P 6700 4850
-AR Path="/6183FAE6/625CAD37/625F8C2E" Ref="R224"  Part="1"
-AR Path="/6183FAE6/6261206B/625F8C2E" Ref="R227"  Part="1"
-F 0 "R227" V 6905 4850 50  0000 C CNN
+AR Path="/6183FAE6/625CAD37/625F8C2E" Ref="R253"  Part="1"
+AR Path="/6183FAE6/6261206B/625F8C2E" Ref="R256"  Part="1"
+F 0 "R256" V 6905 4850 50  0000 C CNN
 F 1 "200" V 6814 4850 50  0000 C CNN
 F 2 "Resistor_SMD:R_0603_1608Metric" V 6740 4840 50  0001 C CNN

Commit message: Driver board: integrated DIN 41612 backplane connector, and made a dedicated parity inhibit sheet with a different set resistor value.
Parts:
- renumbered D136 to D128, D137 to D129, D138 to D130, D139 to D131, D140 to D132, D141 to D133, D142 to D134, D143 to D135, D144 to D136, D145 to D137, D146 to D138, R251 to R243, R252 to R244, R253 to R245
Changed lines of the file:
@@
 P 4900 3150
 AR Path="/6183FAE6/625DC856" Ref="D?"  Part="1"
-AR Path="/6183FAE6/625CAD37/625DC856" Ref="D136"  Part="1"
-AR Path="/6183FAE6/6261206B/625DC856" Ref="D147"  Part="1"
-F 0 "D147" V 4946 3070 50  0000 R CNN
+AR Path="/6183FAE6/625CAD37/625DC856" Ref="D128"  Part="1"
+AR Path="/6183FAE6/6261206B/625DC856" Ref="D139"  Part="1"
+F 0 "D139" V 4946 3070 50  0000 R CNN
 F 1 "1N4148" V 4855 3070 50  0000 R CNN
 F 2 "Diode_SMD:D_SOD-323" H 4900 3150 50  0001 C CNN
@@
 P 5350 3150
 AR Path="/6183FAE6/625DC85D" Ref="D?"  Part="1"
-AR Path="/6183FAE6/625CAD37/625DC85D" Ref="D139"  Part="1"
-AR Path="/6183FAE6/6261206B/625DC85D" Ref="D150"  Part="1"
-F 0 "D150" V 5396 3070 50  0000 R CNN
+AR Path="/6183FAE6/625CAD37/625DC85D" Ref="D131"  Part="1"
+AR Path="/6183FAE6/6261206B/625DC85D" Ref="D142"  Part="1"
+F 0 "D142" V 5396 3070 50  0000 R CNN
 F 1 "1N4148" V 5305 3070 50  0000 R CNN
 F 2 "Diode_SMD:D_SOD-323" H 5350 3150 50  0001 C CNN
@@
 P 5800 3150
 AR Path="/6183FAE6/625DC86B" Ref="D?"  Part="1"
-AR Path="/6183FAE6/625CAD37/625DC86B" Ref="D141"  Part="1"
-AR Path="/6183FAE6/6261206B/625DC86B" Ref="D152"  Part="1"
-F 0 "D152" V 5846 3070 50  0000 R CNN
+AR Path="/6183FAE6/625CAD37/625DC86B" Ref="D133"  Part="1"
+AR Path="/6183FAE6/6261206B/625DC86B" Ref="D144"  Part="1"
+F 0 "D144" V 5846 3070 50  0000 R CNN
 F 1 "1N4148" V 5755 3070 50  0000 R CNN
 F 2 "Diode_SMD:D_SOD-323" H 5800 3150 50  0001 C CNN
@@
 P 6250 3150
 AR Path="/6183FAE6/625DC877" Ref="D?"  Part="1"
-AR Path="/6183FAE6/625CAD37/625DC877" Ref="D144"  Part="1"
-AR Path="/6183FAE6/6261206B/625DC877" Ref="D155"  Part="1"
-F 0 "D155" V 6296 3070 50  0000 R CNN
+AR Path="/6183FAE6/625CAD37/625DC877" Ref="D136"  Part="1"
+AR Path="/6183FAE6/6261206B/625DC877" Ref="D147"  Part="1"
+F 0 "D147" V 6296 3070 50  0000 R CNN
 F 1 "1N4148" V 6205 3070 50  0000 R CNN
 F 2 "Diode_SMD:D_SOD-323" H 6250 3150 50  0001 C CNN
@@
 P 4900 3900
 AR Path="/6183FAE6/625DF9CF" Ref="D?"  Part="1"
-AR Path="/6183FAE6/625CAD37/625DF9CF" Ref="D137"  Part="1"
-AR Path="/6183FAE6/6261206B/625DF9CF" Ref="D148"  Part="1"
-F 0 "D148" V 4946 3820 50  0000 R CNN
+AR Path="/6183FAE6/625CAD37/625DF9CF" Ref="D129"  Part="1"
+AR Path="/6183FAE6/6261206B/625DF9CF" Ref="D140"  Part="1"
+F 0 "D140" V 4946 3820 50  0000 R CNN
 F 1 "1N4148" V 4855 3820 50  0000 R CNN
 F 2 "Diode_SMD:D_SOD-323" H 4900 3900 50  0001 C CNN
@@
 P 5350 3900
 AR Path="/6183FAE6/625DF9EA" Ref="D?"  Part="1"
-AR Path="/6183FAE6/625CAD37/625DF9EA" Ref="D140"  Part="1"
-AR Path="/6183FAE6/6261206B/625DF9EA" Ref="D151"  Part="1"
-F 0 "D151" V 5396 3820 50  0000 R CNN
+AR Path="/6183FAE6/625CAD37/625DF9EA" Ref="D132"  Part="1"
+AR Path="/6183FAE6/6261206B/625DF9EA" Ref="D143"  Part="1"
+F 0 "D143" V 5396 3820 50  0000 R CNN
 F 1 "1N4148" V 5305 3820 50  0000 R CNN
 F 2 "Diode_SMD:D_SOD-323" H 5350 3900 50  0001 C CNN
@@
 P 5800 3900
 AR Path="/6183FAE6/625DF9F8" Ref="D?"  Part="1"
-AR Path="/6183FAE6/625CAD37/625DF9F8" Ref="D142"  Part="1"
-AR Path="/6183FAE6/6261206B/625DF9F8" Ref="D153"  Part="1"
-F 0 "D153" V 5846 3820 50  0000 R CNN
+AR Path="/6183FAE6/625CAD37/625DF9F8" Ref="D134"  Part="1"
+AR Path="/6183FAE6/6261206B/625DF9F8" Ref="D145"  Part="1"
+F 0 "D145" V 5846 3820 50  0000 R CNN
 F 1 "1N4148" V 5755 3820 50  0000 R CNN
 F 2 "Diode_SMD:D_SOD-323" H 5800 3900 50  0001 C CNN
@@
 P 6250 3900
 AR Path="/6183FAE6/625DFA06" Ref="D?"  Part="1"
-AR Path="/6183FAE6/625CAD37/625DFA06" Ref="D145"  Part="1"
-AR Path="/6183FAE6/6261206B/625DFA06" Ref="D156"  Part="1"
-F 0 "D156" V 6296 3820 50  0000 R CNN
+AR Path="/6183FAE6/625CAD37/625DFA06" Ref="D137"  Part="1"
+AR Path="/6183FAE6/6261206B/625DFA06" Ref="D148"  Part="1"
+F 0 "D148" V 6296 3820 50  0000 R CNN
 F 1 "1N4148" V 6205 3820 50  0000 R CNN
 F 2 "Diode_SMD:D_SOD-323" H 6250 3900 50  0001 C CNN
@@
 P 5050 4650
 AR Path="/6183FAE6/625E4460" Ref="D?"  Part="1"
-AR Path="/6183FAE6/625CAD37/625E4460" Ref="D138"  Part="1"
-AR Path="/6183FAE6/6261206B/625E4460" Ref="D149"  Part="1"
-F 0 "D149" V 5096 4570 50  0000 R CNN
+AR Path="/6183FAE6/625CAD37/625E4460" Ref="D130"  Part="1"
+AR Path="/6183FAE6/6261206B/625E4460" Ref="D141"  Part="1"
+F 0 "D141" V 5096 4570 50  0000 R CNN
 F 1 "1N4148" V 5005 4570 50  0000 R CNN
 F 2 "Diode_SMD:D_SOD-323" H 5050 4650 50  0001 C CNN
@@
 	5100 5000 5050 5000
 $Comp
-L Device:R_US R251
+L Device:R_US R243
 U 1 1 625E8581
 P 4800 4850
-AR Path="/6183FAE6/625CAD37/625E8581" Ref="R251"  Part="1"
-AR Path="/6183FAE6/6261206B/625E8581" Ref="R254"  Part="1"
-F 0 "R254" V 5005 4850 50  0000 C CNN
+AR Path="/6183FAE6/625CAD37/625E8581" Ref="R243"  Part="1"
+AR Path="/6183FAE6/6261206B/625E8581" Ref="R246"  Part="1"
+F 0 "R246" V 5005 4850 50  0000 C CNN
 F 1 "200" V 4914 4850 50  0000 C CNN
 F 2 "Resistor_SMD:R_0603_1608Metric" V 4840 4840 50  0001 C CNN
@@
 P 6000 4650
 AR Path="/6183FAE6/625F4CF1" Ref="D?"  Part="1"
-AR Path="/6183FAE6/625CAD37/625F4CF1" Ref="D143"  Part="1"
-AR Path="/6183FAE6/6261206B/625F4CF1" Ref="D154"  Part="1"
-F 0 "D154" V 6046 4570 50  0000 R CNN
+AR Path="/6183FAE6/625CAD37/625F4CF1" Ref="D135"  Part="1"
+AR Path="/6183FAE6/6261206B/625F4CF1" Ref="D146"  Part="1"
+F 0 "D146" V 6046 4570 50  0000 R CNN
 F 1 "1N4148" V 5955 4570 50  0000 R CNN
 F 2 "Diode_SMD:D_SOD-323" H 6000 4650 50  0001 C CNN
@@
 	6050 5000 6000 5000
 $Comp
-L Device:R_US R252
+L Device:R_US R244
 U 1 1 625F4D0E
 P 5750 4850
-AR Path="/6183FAE6/625CAD37/625F4D0E" Ref="R252"  Part="1"
-AR Path="/6183FAE6/6261206B/625F4D0E" Ref="R255"  Part="1"
-F 0 "R255" V 5955 4850 50  0000 C CNN
+AR Path="/6183FAE6/625CAD37/625F4D0E" Ref="R244"  Part="1"
+AR Path="/6183FAE6/6261206B/625F4D0E" Ref="R247"  Part="1"
+F 0 "R247" V 5955 4850 50  0000 C CNN
 F 1 "200" V 5864 4850 50  0000 C CNN
 F 2 "Resistor_SMD:R_0603_1608Metric" V 5790 4840 50  0001 C CNN
@@
 P 6950 4650
 AR Path="/6183FAE6/625F8C11" Ref="D?"  Part="1"
-AR Path="/6183FAE6/625CAD37/625F8C11" Ref="D146"  Part="1"
-AR Path="/6183FAE6/6261206B/625F8C11" Ref="D157"  Part="1"
-F 0 "D157" V 6996 4570 50  0000 R CNN
+AR Path="/6183FAE6/625CAD37/625F8C11" Ref="D138"  Part="1"
+AR Path="/6183FAE6/6261206B/625F8C11" Ref="D149"  Part="1"
+F 0 "D149" V 6996 4570 50  0000 R CNN
 F 1 "1N4148" V 6905 4570 50  0000 R CNN
 F 2 "Diode_SMD:D_SOD-323" H 6950 4650 50  0001 C CNN
@@
 	7000 5000 6950 5000
 $Comp
-L Device:R_US R253
+L Device:R_US R245
 U 1 1 625F8C2E
 P 6700 4850
-AR Path="/6183FAE6/625CAD37/625F8C2E" Ref="R253"  Part="1"
-AR Path="/6183FAE6/6261206B/625F8C2E" Ref="R256"  Part="1"
-F 0 "R256" V 6905 4850 50  0000 C CNN
+AR Path="/6183FAE6/625CAD37/625F8C2E" Ref="R245"  Part="1"
+AR Path="/6183FAE6/6261206B/625F8C2E" Ref="R248"  Part="1"
+F 0 "R248" V 6905 4850 50  0000 C CNN
 F 1 "200" V 6814 4850 50  0000 C CNN
 F 2 "Resistor_SMD:R_0603_1608Metric" V 6740 4840 50  0001 C CNN

Commit message: Driver board: largely fleshed out part selection
Parts:
- D128, D129, D130, D131, D132, D133, D134, D135, D136, D137, D138: Digikey (none) -> https://www.digikey.com/en/products/detail/smc-diode-soluti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; Part Number (none) -> 1N4148WSTR
Changed lines of the file:
@@
 $Descr A4 11693 8268
 encoding utf-8
-Sheet 60 64
+Sheet 52 64
 Title ""
 Date ""
@@
 AR Path="/6183FAE6/625CAD37/625DC856" Ref="D128"  Part="1"
 AR Path="/6183FAE6/6261206B/625DC856" Ref="D139"  Part="1"
-F 0 "D139" V 4946 3070 50  0000 R CNN
+F 0 "D128" V 4946 3070 50  0000 R CNN
 F 1 "1N4148" V 4855 3070 50  0000 R CNN
 F 2 "Diode_SMD:D_SOD-323" H 4900 3150 50  0001 C CNN
 F 3 "~" H 4900 3150 50  0001 C CNN
+F 4 "1N4148WSTR" V 4900 3150 50  0001 C CNN "Part Number"
+F 5 "https://www.digikey.com/en/products/detail/smc-diode-solutions/1N4148WSTR/6022449" V 4900 3150 50  0001 C CNN "Digikey"
 	1    4900 3150
 	0    -1   -1   0
@@
 AR Path="/6183FAE6/625CAD37/625DC85D" Ref="D131"  Part="1"
 AR Path="/6183FAE6/6261206B/625DC85D" Ref="D142"  Part="1"
-F 0 "D142" V 5396 3070 50  0000 R CNN
+F 0 "D131" V 5396 3070 50  0000 R CNN
 F 1 "1N4148" V 5305 3070 50  0000 R CNN
 F 2 "Diode_SMD:D_SOD-323" H 5350 3150 50  0001 C CNN
 F 3 "~" H 5350 3150 50  0001 C CNN
+F 4 "1N4148WSTR" V 4900 3150 50  0001 C CNN "Part Number"
+F 5 "https://www.digikey.com/en/products/detail/smc-diode-solutions/1N4148WSTR/6022449" V 4900 3150 50  0001 C CNN "Digikey"
 	1    5350 3150
 	0    -1   -1   0
@@
 AR Path="/6183FAE6/625CAD37/625DC86B" Ref="D133"  Part="1"
 AR Path="/6183FAE6/6261206B/625DC86B" Ref="D144"  Part="1"
-F 0 "D144" V 5846 3070 50  0000 R CNN
+F 0 "D133" V 5846 3070 50  0000 R CNN
 F 1 "1N4148" V 5755 3070 50  0000 R CNN
 F 2 "Diode_SMD:D_SOD-323" H 5800 3150 50  0001 C CNN
 F 3 "~" H 5800 3150 50  0001 C CNN
+F 4 "1N4148WSTR" V 4900 3150 50  0001 C CNN "Part Number"
+F 5 "https://www.digikey.com/en/products/detail/smc-diode-solutions/1N4148WSTR/6022449" V 4900 3150 50  0001 C CNN "Digikey"
 	1    5800 3150
 	0    -1   -1   0
@@
 AR Path="/6183FAE6/625CAD37/625DC877" Ref="D136"  Part="1"
 AR Path="/6183FAE6/6261206B/625DC877" Ref="D147"  Part="1"
-F 0 "D147" V 6296 3070 50  0000 R CNN
+F 0 "D136" V 6296 3070 50  0000 R CNN
 F 1 "1N4148" V 6205 3070 50  0000 R CNN
 F 2 "Diode_SMD:D_SOD-323" H 6250 3150 50  0001 C CNN
 F 3 "~" H 6250 3150 50  0001 C CNN
+F 4 "1N4148WSTR" V 4900 3150 50  0001 C CNN "Part Number"
+F 5 "https://www.digikey.com/en/products/detail/smc-diode-solutions/1N4148WSTR/6022449" V 4900 3150 50  0001 C CNN "Digikey"
 	1    6250 3150
 	0    -1   -1   0
@@
 AR Path="/6183FAE6/625CAD37/625DF9CF" Ref="D129"  Part="1"
 AR Path="/6183FAE6/6261206B/625DF9CF" Ref="D140"  Part="1"
-F 0 "D140" V 4946 3820 50  0000 R CNN
+F 0 "D129" V 4946 3820 50  0000 R CNN
 F 1 "1N4148" V 4855 3820 50  0000 R CNN
 F 2 "Diode_SMD:D_SOD-323" H 4900 3900 50  0001 C CNN
 F 3 "~" H 4900 3900 50  0001 C CNN
+F 4 "1N4148WSTR" V 4900 3150 50  0001 C CNN "Part Number"
+F 5 "https://www.digikey.com/en/products/detail/smc-diode-solutions/1N4148WSTR/6022449" V 4900 3150 50  0001 C CNN "Digikey"
 	1    4900 3900
 	0    -1   -1   0
@@
 AR Path="/6183FAE6/625CAD37/625DF9EA" Ref="D132"  Part="1"
 AR Path="/6183FAE6/6261206B/625DF9EA" Ref="D143"  Part="1"
-F 0 "D143" V 5396 3820 50  0000 R CNN
+F 0 "D132" V 5396 3820 50  0000 R CNN
 F 1 "1N4148" V 5305 3820 50  0000 R CNN
 F 2 "Diode_SMD:D_SOD-323" H 5350 3900 50  0001 C CNN
 F 3 "~" H 5350 3900 50  0001 C CNN
+F 4 "1N4148WSTR" V 4900 3150 50  0001 C CNN "Part Number"
+F 5 "https://www.digikey.com/en/products/detail/smc-diode-solutions/1N4148WSTR/6022449" V 4900 3150 50  0001 C CNN "Digikey"
 	1    5350 3900
 	0    -1   -1   0
@@
 AR Path="/6183FAE6/625CAD37/625DF9F8" Ref="D134"  Part="1"
 AR Path="/6183FAE6/6261206B/625DF9F8" Ref="D145"  Part="1"
-F 0 "D145" V 5846 3820 50  0000 R CNN
+F 0 "D134" V 5846 3820 50  0000 R CNN
 F 1 "1N4148" V 5755 3820 50  0000 R CNN
 F 2 "Diode_SMD:D_SOD-323" H 5800 3900 50  0001 C CNN
 F 3 "~" H 5800 3900 50  0001 C CNN
+F 4 "1N4148WSTR" V 4900 3150 50  0001 C CNN "Part Number"
+F 5 "https://www.digikey.com/en/products/detail/smc-diode-solutions/1N4148WSTR/6022449" V 4900 3150 50  0001 C CNN "Digikey"
 	1    5800 3900
 	0    -1   -1   0
@@
 AR Path="/6183FAE6/625CAD37/625DFA06" Ref="D137"  Part="1"
 AR Path="/6183FAE6/6261206B/625DFA06" Ref="D148"  Part="1"
-F 0 "D148" V 6296 3820 50  0000 R CNN
+F 0 "D137" V 6296 3820 50  0000 R CNN
 F 1 "1N4148" V 6205 3820 50  0000 R CNN
 F 2 "Diode_SMD:D_SOD-323" H 6250 3900 50  0001 C CNN
 F 3 "~" H 6250 3900 50  0001 C CNN
+F 4 "1N4148WSTR" V 4900 3150 50  0001 C CNN "Part Number"
+F 5 "https://www.digikey.com/en/products/detail/smc-diode-solutions/1N4148WSTR/6022449" V 4900 3150 50  0001 C CNN "Digikey"
 	1    6250 3900
 	0    -1   -1   0
@@
 AR Path="/6183FAE6/625CAD37/625E4460" Ref="D130"  Part="1"
 AR Path="/6183FAE6/6261206B/625E4460" Ref="D141"  Part="1"
-F 0 "D141" V 5096 4570 50  0000 R CNN
+F 0 "D130" V 5096 4570 50  0000 R CNN
 F 1 "1N4148" V 5005 4570 50  0000 R CNN
 F 2 "Diode_SMD:D_SOD-323" H 5050 4650 50  0001 C CNN
 F 3 "~" H 5050 4650 50  0001 C CNN
+F 4 "1N4148WSTR" V 4900 3150 50  0001 C CNN "Part Number"
+F 5 "https://www.digikey.com/en/products/detail/smc-diode-solutions/1N4148WSTR/6022449" V 4900 3150 50  0001 C CNN "Digikey"
 	1    5050 4650
 	0    -1   -1   0
@@
 AR Path="/6183FAE6/625CAD37/625E8581" Ref="R243"  Part="1"
 AR Path="/6183FAE6/6261206B/625E8581" Ref="R246"  Part="1"
-F 0 "R246" V 5005 4850 50  0000 C CNN
+F 0 "R243" V 5005 4850 50  0000 C CNN
 F 1 "200" V 4914 4850 50  0000 C CNN
 F 2 "Resistor_SMD:R_0603_1608Metric" V 4840 4840 50  0001 C CNN
@@
 AR Path="/6183FAE6/625CAD37/625F4CF1" Ref="D135"  Part="1"
 AR Path="/6183FAE6/6261206B/625F4CF1" Ref="D146"  Part="1"
-F 0 "D146" V 6046 4570 50  0000 R CNN
+F 0 "D135" V 6046 4570 50  0000 R CNN
 F 1 "1N4148" V 5955 4570 50  0000 R CNN
 F 2 "Diode_SMD:D_SOD-323" H 6000 4650 50  0001 C CNN
 F 3 "~" H 6000 4650 50  0001 C CNN
+F 4 "1N4148WSTR" V 4900 3150 50  0001 C CNN "Part Number"
+F 5 "https://www.digikey.com/en/products/detail/smc-diode-solutions/1N4148WSTR/6022449" V 4900 3150 50  0001 C CNN "Digikey"
 	1    6000 4650
 	0    -1   -1   0
@@
 AR Path="/6183FAE6/625CAD37/625F4D0E" Ref="R244"  Part="1"
 AR Path="/6183FAE6/6261206B/625F4D0E" Ref="R247"  Part="1"
-F 0 "R247" V 5955 4850 50  0000 C CNN
+F 0 "R244" V 5955 4850 50  0000 C CNN
 F 1 "200" V 5864 4850 50  0000 C CNN
 F 2 "Resistor_SMD:R_0603_1608Metric" V 5790 4840 50  0001 C CNN
@@
 AR Path="/6183FAE6/625CAD37/625F8C11" Ref="D138"  Part="1"
 AR Path="/6183FAE6/6261206B/625F8C11" Ref="D149"  Part="1"
-F 0 "D149" V 6996 4570 50  0000 R CNN
+F 0 "D138" V 6996 4570 50  0000 R CNN
 F 1 "1N4148" V 6905 4570 50  0000 R CNN
 F 2 "Diode_SMD:D_SOD-323" H 6950 4650 50  0001 C CNN
 F 3 "~" H 6950 4650 50  0001 C CNN
+F 4 "1N4148WSTR" V 4900 3150 50  0001 C CNN "Part Number"
+F 5 "https://www.digikey.com/en/products/detail/smc-diode-solutions/1N4148WSTR/6022449" V 4900 3150 50  0001 C CNN "Digikey"
 	1    6950 4650
 	0    -1   -1   0
@@
 AR Path="/6183FAE6/625CAD37/625F8C2E" Ref="R245"  Part="1"
 AR Path="/6183FAE6/6261206B/625F8C2E" Ref="R248"  Part="1"
-F 0 "R248" V 6905 4850 50  0000 C CNN
+F 0 "R245" V 6905 4850 50  0000 C CNN
 F 1 "200" V 6814 4850 50  0000 C CNN
 F 2 "Resistor_SMD:R_0603_1608Metric" V 6740 4840 50  0001 C CNN
