File: boards/driver/sense_amps.sch (KiCad schematic (older format))
At the start: 5 parts, among them U1 AD1582BRTZ

Commit message: Driver board: integrated DIN 41612 backplane connector, and made a dedicated parity inhibit sheet with a different set resistor value.
Parts:
- R1, R2: footprint (none) -> Resistor_SMD:R_0603_1608Metric
- U1: footprint (none) -> Package_TO_SOT_SMD:SOT-23
Changed lines of the file:
@@
 F 0 "U1" H 8450 3815 50  0000 C CNN
 F 1 "AD1582BRTZ" H 8450 3724 50  0000 C CNN
-F 2 "" H 8550 3450 50  0001 C CNN
+F 2 "Package_TO_SOT_SMD:SOT-23" H 8550 3450 50  0001 C CNN
 F 3 "" H 8550 3450 50  0001 C CNN
 	1    8450 3450
@@
 F 0 "R1" H 9418 3646 50  0000 L CNN
 F 1 "1.27k" H 9418 3555 50  0000 L CNN
-F 2 "" V 9390 3590 50  0001 C CNN
+F 2 "Resistor_SMD:R_0603_1608Metric" V 9390 3590 50  0001 C CNN
 F 3 "~" H 9350 3600 50  0001 C CNN
 	1    9350 3600
@@
 F 0 "R2" H 9418 4046 50  0000 L CNN
 F 1 "249" H 9418 3955 50  0000 L CNN
-F 2 "" V 9390 3990 50  0001 C CNN
+F 2 "Resistor_SMD:R_0603_1608Metric" V 9390 3990 50  0001 C CNN
 F 3 "~" H 9350 4000 50  0001 C CNN
 	1    9350 4000

Commit message: Driver board: largely fleshed out part selection
Parts:
- C1: footprint (none) -> Capacitor_SMD:C_0805_2012Metric; Digikey (none) -> https://www.digikey.com/en/products/detail/samsung-electro-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; Part Number (none) -> CL21B475KOFNFNE; Rating (none) -> 16V; Tolerance (none) -> 10%
- C2: value 1uF -> 1.0uF; footprint (none) -> Capacitor_SMD:C_0603_1608Metric; Digikey (none) -> https://www.digikey.com/en/products/detail/samsung-electro-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; Part Number (none) -> CL10B105KP8NNNC; Rating (none) -> 10V; Tolerance (none) -> 10%
- U1: Digikey (none) -> https://www.digikey.com/en/products/detail/analog-devices-i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; Part Number (none) -> AD1582BRTZ
Changed lines of the file:
@@
 F 2 "Package_TO_SOT_SMD:SOT-23" H 8550 3450 50  0001 C CNN
 F 3 "" H 8550 3450 50  0001 C CNN
+F 4 "https://www.digikey.com/en/products/detail/analog-devices-inc/AD1582BRTZ-REEL7/750867" H 8450 3450 50  0001 C CNN "Digikey"
+F 5 "AD1582BRTZ" H 8450 3450 50  0001 C CNN "Part Number"
 	1    8450 3450
 	1    0    0    -1
@@
 F 0 "C1" H 7686 3504 50  0000 R CNN
 F 1 "4.7uF" H 7686 3595 50  0000 R CNN
-F 2 "" H 7838 3400 50  0001 C CNN
+F 2 "Capacitor_SMD:C_0805_2012Metric" H 7838 3400 50  0001 C CNN
 F 3 "~" H 7800 3550 50  0001 C CNN
+F 4 "https://www.digikey.com/en/products/detail/samsung-electro-mechanics/CL21B475KOFNFNE/3888628" H 7800 3550 50  0001 C CNN "Digikey"
+F 5 "CL21B475KOFNFNE" H 7800 3550 50  0001 C CNN "Part Number"
+F 6 "16V" H 7600 3700 50  0000 C CNN "Rating"
+F 7 "10%" H 7600 3800 50  0000 C CNN "Tolerance"
 	1    7800 3550
 	1    0    0    1
@@
 P 8850 3600
 F 0 "C2" H 8965 3646 50  0000 L CNN
-F 1 "1uF" H 8965 3555 50  0000 L CNN
-F 2 "" H 8888 3450 50  0001 C CNN
+F 1 "1.0uF" H 8965 3555 50  0000 L CNN
+F 2 "Capacitor_SMD:C_0603_1608Metric" H 8888 3450 50  0001 C CNN
 F 3 "~" H 8850 3600 50  0001 C CNN
+F 4 "https://www.digikey.com/en/products/detail/samsung-electro-mechanics/CL10B105KP8NNNC/3887604" H 8850 3600 50  0001 C CNN "Digikey"
+F 5 "" H 8850 3600 50  0001 C CNN "ESR"
+F 6 "CL10B105KP8NNNC" H 8850 3600 50  0001 C CNN "Part Number"
+F 7 "10V" H 9050 3450 50  0000 C CNN "Rating"
+F 8 "10%" H 9050 3350 50  0000 C CNN "Tolerance"
 	1    8850 3600
 	1    0    0    -1
