File: boards/driver/driver.kicad_pcb (KiCad board)
At the start: 2 copper layers, 228.6 x 116.8 mm, 646 parts, among them J1 Barrel_Jack_Switch, J2 Conn_01x24, J3 Conn_02x06_Top_Bottom, J4 Conn_01x24, J5 Conn_01x24, J6 Conn_01x24, J7 Conn_01x24, J8 Conn_01x24, Q1 MMBT2222, Q10 MMBT2222, Q11 MMBT2907, Q12 MMBT2222, Q13 MMBT2907, Q14 MMBT2222, Q15 MMBT2907, Q16 MMBT2222, Q17 MMBT2907, Q18 MMBT2222, Q19 MMBT2907, Q2 MMBT2907, Q20 MMBT2222, Q21 MMBT2907, Q22 MMBT2222, Q23 MMBT2907, Q24 MMBT2222, Q25 MMBT2907, Q26 MMBT2222, Q27 MMBT2907, Q28 MMBT2222, Q29 MMBT2222, Q3 MMBT2222, Q30 MMBT2222, Q31 MMBT2222, Q32 MMBT2222, Q33 MMBT2222, Q34 MMBT2222, Q35 MMBT2222, Q36 MMBT2222, Q37 MMBT2222, Q38 MMBT2222, Q39 MMBT2222, Q4 MMBT2222, Q40 MMBT2222, Q41 MMBT2222, Q42 MMBT2222, Q43 MMBT2222, Q44 MMBT2222, Q45 MMBT2222, Q46 MMBT2222, Q47 MMBT2222, Q48 MMBT2222, Q49 MMBT2222, Q5 MMBT2907, Q50 MMBT2222, Q51 MMBT2222, Q52 MMBT2222, Q53 MMBT2222, Q54 MMBT2222, Q55 MMBT2222, Q56 MMBT2222, Q57 MMBT2222, Q58 MMBT2222, Q59 MMBT2222, Q6 MMBT2222, Q60 MMBT2222, Q61 MMBT2907, Q62 MMBT2222, Q63 MMBT2222, Q64 MMBT2907, Q65 MMBT2222, Q66 MMBT2222, Q67 MMBT2907, Q68 MMBT2222, Q69 MMBT2222, Q7 MMBT2907, Q70 MMBT2222, Q71 MMBT2907, Q72 MMBT2222, Q73 MMBT2222, Q74 MMBT2222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

Commit message: Driver board: integrated DIN 41612 backplane connector, and made a dedicated parity inhibit sheet with a different set resistor value.
Parts:
- removed J6, J7, J8: Conn_01x24, Connector_PinHeader_1.00mm:PinHeader_1x24_P1.00mm_Vertical
- added R1: 1.27k, Resistor_SMD:R_0603_1608Metric, F.Cu at (177.0, -1.54)
- added R2: 249, Resistor_SMD:R_0603_1608Metric, F.Cu at (177.0, 0.97)
- added U1: AD1582BRTZ, Package_TO_SOT_SMD:SOT-23, F.Cu at (172.8, -0.52)
- J5: value Conn_01x24 -> DIN41612_03x32_C; footprint Connector_PinHeader_1.00mm:PinHeader_1x24_P1.00mm_Vertical -> Connector_DIN:DIN41612_C_3x32_Male_Horizontal_THT
- L17, L18: value 2.2uH -> 3.9uH
- L29, L30: value 3.9uH -> 8.2uH
- L37, L38: value 8.2uH -> 2.2uH
- Q57, Q60, Q63: value MMBT2222 -> MMBT2907
- Q61, Q64, Q87: value MMBT2907 -> MMBT2222
- R180: value 390 -> 470
- R181: value 3.9 -> 2k
- R182: value NOM -> 750
- R183: value 1k -> 2k
- R184: value 390 -> 1k
- R185: value 3.9 -> 470
- R186: value NOM -> 2k
- R187: value 1k -> 750
- R188: value 470 -> 2k
- R189: value 2k -> 1k
- R190: value 750 -> 1k
- R191: value 2k -> 5.1k
- R192: value 1k -> 5.1k
- R193: value 470 -> 27
- R194, R196: value 2k -> 7.5
- R195: value 750 -> NOM
- R197, R206, R215, R224, R233, R242: value 1k -> NOM
- R199, R208, R217, R226, R235: value 5.1k -> 1k
- R201, R210, R219, R228, R237: value 27 -> 5.1k
- R202, R211, R220, R229, R238: value 7.5 -> 27
- R203, R205, R212, R214, R221, R223, R230, R232, R239, R241: value NOM -> 7.5
- R204, R213, R222, R231, R240: value 7.5 -> NOM
- R243: value 1k -> 200
- R244, R245: value 5.1k -> 200
- R246: value 27 -> 200
- R247: value 7.5 -> 200
- R248: value NOM -> 200
- R249: value 7.5 -> 3k
- R250: value NOM -> 3k
- R251, R255: value 200 -> 1k
- R252, R256: value 200 -> 390
- R253: value 200 -> 2.2
- R254: value 200 -> NOM
- R257: value 3k -> 2.2
- R258: value 3k -> NOM
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Connections:
- D100 pad 1: GND -> Net-(D100-Pad1)
- D100 pad 2: Net-(D100-Pad2) -> /Rope Drivers/BPLIZ2
- D101 pad 2: /Rope Drivers/BPLIZ1 -> Net-(D100-Pad1)
- D103 pad 2: Net-(D102-Pad1) -> Net-(D103-Pad2)
- D104 pad 2: Net-(D104-Pad2) -> Net-(D103-Pad1)
- D106 pad 1: Net-(D106-Pad1) -> GND
- D107 pad 1: GND -> Net-(D107-Pad1)
- D107 pad 2: Net-(D106-Pad1) -> /Rope Drivers/BPLIZ1
- D108 pad 2: /Rope Drivers/BPLIZ2 -> Net-(D107-Pad1)
- D110 pad 2: Net-(D109-Pad1) -> Net-(D110-Pad2)
- D111 pad 2: Net-(D111-Pad2) -> Net-(D110-Pad1)
- D113 pad 1: Net-(D113-Pad1) -> GND
- D114 pad 1: GND -> Net-(D114-Pad1)
- D114 pad 2: Net-(D113-Pad1) -> /Rope Drivers/BPLIZ2
- D115 pad 2: /Rope Drivers/BPLIZ1 -> Net-(D114-Pad1)
- D117 pad 2: Net-(D116-Pad1) -> Net-(D117-Pad2)
- D118 pad 2: Net-(D118-Pad2) -> Net-(D117-Pad1)
- D120 pad 1: Net-(D120-Pad1) -> GND
- D121 pad 1: GND -> Net-(D121-Pad1)
- D121 pad 2: Net-(D120-Pad1) -> /Rope Drivers/BPLIZ1
- D122 pad 2: /Rope Drivers/BPLIZ2 -> Net-(D121-Pad1)
- D124 pad 2: Net-(D123-Pad1) -> Net-(D124-Pad2)
- D125 pad 2: Net-(D125-Pad2) -> Net-(D124-Pad1)
- D127 pad 1: Net-(D127-Pad1) -> GND
- D128 pad 1: GND -> /Connector/RFD1
- D128 pad 2: Net-(D127-Pad1) -> /Rope Drivers/BPLMX1
- D129 pad 1: Net-(D129-Pad1) -> /Connector/RFD3
- D129 pad 2: /Rope Drivers/BPLIZ1 -> /Rope Drivers/BPLMX2
- D130 pad 1: Net-(D130-Pad1) -> /Connector/RSTRD4
- D130 pad 2: Net-(D129-Pad1) -> /Rope Drivers/BPLMX3
- D131 pad 1: Net-(D131-Pad1) -> /Connector/RCD1
- D131 pad 2: Net-(D130-Pad1) -> /Rope Drivers/BPLMX1
- D132 pad 1: Net-(D132-Pad1) -> /Connector/RCD3
- D132 pad 2: Net-(D132-Pad2) -> /Rope Drivers/BPLMX2
- D133 pad 1: Net-(D133-Pad1) -> /Connector/RFD2
- D133 pad 2: Net-(D132-Pad1) -> /Rope Drivers/BPLMX1
- D134 pad 1: Net-(D134-Pad1) -> /Connector/RFD4
- D134 pad 2: Net-(D133-Pad1) -> /Rope Drivers/BPLMX2
- D135 pad 1: GND -> /Connector/RSTRD3
- D135 pad 2: Net-(D134-Pad1) -> /Rope Drivers/BPLMX3
- D136 pad 1: /Connector/RFD1 -> /Connector/RCD2
- D137 pad 1: /Connector/RFD3 -> /Connector/RCD4
- D138 pad 1: /Connector/RSTRD4 -> /Connector/SETRN1
- D139 pad 1: /Connector/RCD1 -> /Connector/RFD5
- D140 pad 1: /Connector/RCD3 -> /Connector/RFD7
- D141 pad 1: /Connector/RFD2 -> /Connector/RSTRD2
- D141 pad 2: /Rope Drivers/BPLMX1 -> /Rope Drivers/BPLMX3
- D142 pad 1: /Connector/RFD4 -> /Connector/RCD5
- D142 pad 2: /Rope Drivers/BPLMX2 -> /Rope Drivers/BPLMX1
- D143 pad 1: /Connector/RSTRD3 -> /Connector/RCD7
- D143 pad 2: /Rope Drivers/BPLMX3 -> /Rope Drivers/BPLMX2
- D144 pad 1: /Connector/RCD2 -> /Connector/RFD6
- D145 pad 1: /Connector/RCD4 -> /Connector/RFD8
- D146 pad 1: /Connector/SETRN1 -> /Connector/RSTRD1
- D147 pad 1: /Connector/RFD5 -> /Connector/RCD6
- D148 pad 1: /Connector/RFD7 -> /Connector/RCD8
- D149 pad 1: /Connector/RSTRD2 -> /Connector/SETRN2
- D150 pad 1: /Connector/RCD5 -> GND
- D150 pad 2: /Rope Drivers/BPLMX1 -> GND
- D151 pad 1: /Connector/RCD7 -> GND
- D151 pad 2: /Rope Drivers/BPLMX2 -> GND
- D152 pad 1: /Connector/RFD6 -> Net-(D152-Pad1)
- D152 pad 2: /Rope Drivers/BPLMX1 -> Net-(D152-Pad2)
- D153 pad 1: /Connector/RFD8 -> Net-(D153-Pad1)
- D153 pad 2: /Rope Drivers/BPLMX2 -> Net-(D152-Pad1)
- D154 pad 1: /Connector/RSTRD1 -> Net-(D154-Pad1)
- D154 pad 2: /Rope Drivers/BPLMX3 -> Net-(D153-Pad1)
- D155 pad 1: /Connector/RCD6 -> GND
- D155 pad 2: /Rope Drivers/BPLMX1 -> Net-(D154-Pad1)
- D156 pad 1: /Connector/RCD8 -> Net-(D156-Pad1)
- D156 pad 2: /Rope Drivers/BPLMX2 -> Net-(D156-Pad2)
- D157 pad 1: /Connector/SETRN2 -> Net-(D157-Pad1)
- D157 pad 2: /Rope Drivers/BPLMX3 -> Net-(D156-Pad1)
- D158 pad 1: GND -> Net-(D158-Pad1)
- D158 pad 2: GND -> Net-(D157-Pad1)
- D159 pad 2: GND -> Net-(D158-Pad1)
- D86 pad 2: Net-(D86-Pad2) -> /Rope Drivers/BPLIZ2
- D89 pad 1: GND -> Net-(D89-Pad1)
- D89 pad 2: Net-(D88-Pad1) -> Net-(D89-Pad2)
- D90 pad 2: Net-(D90-Pad2) -> Net-(D89-Pad1)
- D92 pad 1: Net-(D92-Pad1) -> GND
- D93 pad 1: GND -> Net-(D93-Pad1)
- D93 pad 2: Net-(D92-Pad1) -> /Rope Drivers/BPLIZ1
- D94 pad 2: /Rope Drivers/BPLIZ2 -> Net-(D93-Pad1)
- D96 pad 2: Net-(D95-Pad1) -> Net-(D96-Pad2)
- D97 pad 2: Net-(D97-Pad2) -> Net-(D96-Pad1)
- D99 pad 1: Net-(D100-Pad2) -> GND
- L17 pad 2: Net-(D88-Pad1) -> GND
- L18 pad 2: Net-(D92-Pad1) -> GND
- L29 pad 1: Net-(L29-Pad1) -> +14V
- L29 pad 2: GND -> /Rope Drivers/BPLIZ1
- L30 pad 1: Net-(L30-Pad1) -> +14V
- L30 pad 2: GND -> /Rope Drivers/BPLIZ2
- L31 pad 2: /Rope Drivers/BPLIZ1 -> /Rope Drivers/BPLMX1
- L32 pad 2: /Rope Drivers/BPLIZ2 -> /Rope Drivers/BPLMX2
- L33 pad 2: /Rope Drivers/BPLMX1 -> /Rope Drivers/BPLMX3
- L34 pad 2: /Rope Drivers/BPLMX2 -> /Rope Drivers/BPLMX1
- L35 pad 2: /Rope Drivers/BPLMX3 -> /Rope Drivers/BPLMX2
- L36 pad 2: /Rope Drivers/BPLMX1 -> /Rope Drivers/BPLMX3
- L37 pad 1: +14V -> Net-(L37-Pad1)
- L37 pad 2: /Rope Drivers/BPLMX2 -> Net-(D154-Pad1)
- L38 pad 1: +14V -> Net-(L38-Pad1)
- L38 pad 2: /Rope Drivers/BPLMX3 -> Net-(D158-Pad1)
- Q29 pad 3: /Connector/XCN8 -> /Connector/XCN7
- Q31 pad 3: /Connector/XCN7 -> /Connector/XCN6
- Q33 pad 3: /Connector/XCN6 -> /Connector/XCN5
- Q35 pad 3: /Connector/XCN5 -> /Connector/XCN4
- Q37 pad 3: /Connector/XCN4 -> /Connector/XCN3
- Q39 pad 3: /Connector/XCN3 -> /Connector/XCN2
- Q41 pad 3: /Connector/XCN2 -> /Connector/XCN1
- Q43 pad 3: /Connector/XCN1 -> /Connector/XFN7
- Q45 pad 3: /Connector/XFN8 -> /Connector/XFN6
- Q47 pad 3: /Connector/XFN7 -> /Connector/XFN5
- Q49 pad 3: /Connector/XFN6 -> /Connector/XFN4
- Q51 pad 3: /Connector/XFN5 -> /Connector/XFN3
- Q53 pad 3: /Connector/XFN4 -> /Connector/XFN2
- Q55 pad 3: /Connector/XFN3 -> /Connector/XFN1
- Q56 pad 3: Net-(D86-Pad2) -> Net-(Q56-Pad3)
- Q57 pad 1: Net-(D86-Pad2) -> Net-(Q57-Pad1)
- Q57 pad 2: Net-(Q57-Pad2) -> /Rope Drivers/BPLIZ2
- Q57 pad 3: /Connector/XFN2 -> Net-(Q57-Pad3)
- Q58 pad 1: Net-(Q58-Pad1) -> Net-(Q57-Pad3)
- Q58 pad 2: GND -> /Rope Drivers/40332A
- Q58 pad 3: Net-(D90-Pad2) -> /Rope Drivers/BPLIZ2
- Q59 pad 1: Net-(D90-Pad2) -> Net-(Q59-Pad1)
- Q59 pad 2: Net-(Q59-Pad2) -> GND
- Q59 pad 3: /Connector/XFN1 -> Net-(Q59-Pad3)
- Q60 pad 2: GND -> /Rope Drivers/BPLIZ1
- Q61 pad 1: Net-(Q61-Pad1) -> Net-(Q60-Pad3)
- Q61 pad 2: /Rope Drivers/BPLIZ2 -> /Rope Drivers/40331A
- Q61 pad 3: Net-(Q61-Pad3) -> /Rope Drivers/BPLIZ1
- Q62 pad 1: Net-(Q61-Pad3) -> Net-(Q62-Pad1)
- Q62 pad 2: /Rope Drivers/40332A -> GND
- Q62 pad 3: /Rope Drivers/BPLIZ2 -> Net-(Q62-Pad3)
- Q63 pad 1: Net-(Q63-Pad1) -> Net-(D88-Pad1)
- Q63 pad 2: GND -> Net-(Q63-Pad2)
- Q63 pad 3: Net-(Q63-Pad3) -> Net-(D89-Pad2)
- Q64 pad 1: Net-(Q64-Pad1) -> Net-(D89-Pad2)
- Q64 pad 2: /Rope Drivers/BPLIZ1 -> Net-(Q64-Pad2)
- Q64 pad 3: Net-(Q64-Pad3) -> /Connector/XRST4
- Q65 pad 1: Net-(Q64-Pad3) -> Net-(D89-Pad2)
- Q65 pad 2: /Rope Drivers/40331A -> Net-(Q65-Pad2)
- Q65 pad 3: /Rope Drivers/BPLIZ1 -> /Connector/XRST4
- Q67 pad 1: Net-(D96-Pad1) -> Net-(D95-Pad1)
- Q67 pad 3: Net-(D97-Pad2) -> Net-(D96-Pad2)
- Q68 pad 1: Net-(D97-Pad2) -> Net-(D96-Pad2)
- Q68 pad 3: /Connector/XRST4 -> /Connector/XRST3
- Q69 pad 1: Net-(D97-Pad2) -> Net-(D96-Pad2)
- Q69 pad 3: /Connector/XRST4 -> /Connector/XRST3
- Q71 pad 1: Net-(D103-Pad1) -> Net-(D102-Pad1)
- Q71 pad 3: Net-(D104-Pad2) -> Net-(D103-Pad2)
- Q72 pad 1: Net-(D104-Pad2) -> Net-(D103-Pad2)
- Q72 pad 3: /Connector/XRST3 -> /Connector/XRST2
- Q73 pad 1: Net-(D104-Pad2) -> Net-(D103-Pad2)
- Q73 pad 3: /Connector/XRST3 -> /Connector/XRST2
- Q75 pad 1: Net-(D110-Pad1) -> Net-(D109-Pad1)
- Q75 pad 3: Net-(D111-Pad2) -> Net-(D110-Pad2)
- Q76 pad 1: Net-(D111-Pad2) -> Net-(D110-Pad2)
- Q76 pad 3: /Connector/XRST2 -> /Connector/XRST1
- Q77 pad 1: Net-(D111-Pad2) -> Net-(D110-Pad2)
- Q77 pad 3: /Connector/XRST2 -> /Connector/XRST1
- Q79 pad 1: Net-(D117-Pad1) -> Net-(D116-Pad1)
- Q79 pad 3: Net-(D118-Pad2) -> Net-(D117-Pad2)
- Q80 pad 1: Net-(D118-Pad2) -> Net-(D117-Pad2)
- Q80 pad 3: /Connector/XRST1 -> /Connector/XSET2
- Q81 pad 1: Net-(D118-Pad2) -> Net-(D117-Pad2)
- Q81 pad 3: /Connector/XRST1 -> /Connector/XSET2
- Q83 pad 1: Net-(D124-Pad1) -> Net-(D123-Pad1)
- Q83 pad 3: Net-(D125-Pad2) -> Net-(D124-Pad2)
- Q84 pad 1: Net-(D125-Pad2) -> Net-(D124-Pad2)
- Q84 pad 3: /Connector/XSET2 -> /Connector/XSET1
- Q85 pad 1: Net-(D125-Pad2) -> Net-(D124-Pad2)
- Q85 pad 3: /Connector/XSET2 -> /Connector/XSET1
- Q86 pad 3: Net-(Q86-Pad3) -> Net-(D152-Pad2)
- Q87 pad 1: Net-(D131-Pad1) -> Net-(D152-Pad2)
- Q87 pad 3: Net-(D132-Pad2) -> /Connector/XFN8
- Q88 pad 1: Net-(D132-Pad2) -> Net-(Q88-Pad1)
- Q88 pad 2: Net-(Q88-Pad2) -> GND
- Q88 pad 3: /Connector/XSET1 -> Net-(D156-Pad2)
- Q89 pad 1: Net-(D132-Pad2) -> Net-(D156-Pad2)
- Q89 pad 3: /Connector/XSET1 -> /Connector/XCN8
- R123 pad 2: /FPGA and Power/~IL8 -> /FPGA and Power/~IL7
- R127 pad 2: /FPGA and Power/~IL7 -> /FPGA and Power/~IL6
- R131 pad 2: /FPGA and Power/~IL6 -> /FPGA and Power/~IL5
- R135 pad 2: /FPGA and Power/~IL5 -> /FPGA and Power/~IL4
- R139 pad 2: /FPGA and Power/~IL4 -> /FPGA and Power/~IL3
- R140 pad 1: /Rope Drivers/40332A -> /Rope Drivers/40331A
- R143 pad 2: /FPGA and Power/~IL3 -> /FPGA and Power/~IL2
- R147 pad 2: /FPGA and Power/~IL2 -> /FPGA and Power/~IL1
- R151 pad 2: /FPGA and Power/~IL1 -> /FPGA and Power/IL7
- R152 pad 1: /Rope Drivers/40331A -> /Rope Drivers/40332A
- R155 pad 2: /FPGA and Power/IL8 -> /FPGA and Power/IL6
- R156 pad 1: /Rope Drivers/40331A -> /Rope Drivers/40332A
- R159 pad 2: /FPGA and Power/IL7 -> /FPGA and Power/IL5
- R163 pad 2: /FPGA and Power/IL6 -> /FPGA and Power/IL4
- R164 pad 1: /Rope Drivers/40332A -> /Rope Drivers/40331A
- R167 pad 2: /FPGA and Power/IL5 -> /FPGA and Power/IL3
- R168 pad 1: /Rope Drivers/40332A -> /Rope Drivers/40331A
- R171 pad 2: /FPGA and Power/IL4 -> /FPGA and Power/IL2
- R175 pad 2: /FPGA and Power/IL3 -> /FPGA and Power/IL1
- R179 pad 2: /FPGA and Power/IL2 -> /FPGA and Power/IHENV
- R180 pad 1: /Rope Drivers/40331A -> /Rope Drivers/BPLIZ2
- R180 pad 2: Net-(D86-Pad2) -> Net-(Q57-Pad1)
- R181 pad 1: Net-(Q57-Pad2) -> Net-(Q57-Pad1)
- R181 pad 2: Net-(R181-Pad2) -> Net-(Q56-Pad3)
- R182 pad 1: Net-(R181-Pad2) -> Net-(Q57-Pad3)
- R182 pad 2: Net-(L17-Pad1) -> GND
- R183 pad 1: Net-(Q58-Pad1) -> /Rope Drivers/40332A
- R183 pad 2: /FPGA and Power/IL1 -> GND
- R184 pad 1: /Rope Drivers/40331A -> Net-(Q59-Pad1)
- R184 pad 2: Net-(D90-Pad2) -> /FPGA and Power/IHENV
- R185 pad 1: Net-(Q59-Pad2) -> /Rope Drivers/BPLIZ1
- R185 pad 2: Net-(R185-Pad2) -> Net-(Q60-Pad1)
- R186 pad 1: Net-(R185-Pad2) -> Net-(Q60-Pad1)
- R186 pad 2: Net-(L18-Pad1) -> Net-(Q59-Pad3)
- R187 pad 1: Net-(Q60-Pad1) -> Net-(Q60-Pad3)
- R187 pad 2: /FPGA and Power/IHENV -> GND
- R188 pad 1: /Rope Drivers/BPLIZ2 -> /Rope Drivers/40331A
- R188 pad 2: Net-(Q61-Pad1) -> GND
- R189 pad 1: Net-(Q61-Pad1) -> Net-(Q62-Pad1)
- R189 pad 2: Net-(Q60-Pad3) -> /FPGA and Power/RESET4
- R190 pad 1: Net-(Q61-Pad3) -> Net-(D88-Pad1)
- R190 pad 2: GND -> Net-(Q62-Pad3)
- R191 pad 1: /Rope Drivers/40332A -> /Rope Drivers/BPLIZ2
- R191 pad 2: GND -> Net-(D88-Pad1)
- R192 pad 1: Net-(Q63-Pad1) -> Net-(D89-Pad2)
- R192 pad 2: /FPGA and Power/IHENV -> GND
- R193 pad 1: /Rope Drivers/BPLIZ1 -> /Rope Drivers/BPLIZ2
- R193 pad 2: Net-(Q64-Pad1) -> Net-(Q63-Pad2)
- R194 pad 1: Net-(Q64-Pad1) -> Net-(Q64-Pad2)
- R194 pad 2: Net-(Q63-Pad3) -> Net-(R194-Pad2)
- R195 pad 1: Net-(Q64-Pad3) -> Net-(R194-Pad2)
- R195 pad 2: GND -> Net-(L17-Pad1)
- R196 pad 1: /Rope Drivers/40331A -> Net-(Q65-Pad2)
- R196 pad 2: GND -> Net-(R196-Pad2)
- R197 pad 1: Net-(Q66-Pad1) -> Net-(R196-Pad2)
- R197 pad 2: /FPGA and Power/RESET4 -> Net-(L18-Pad1)
- R198 pad 1: Net-(D96-Pad1) -> Net-(Q66-Pad1)
- R198 pad 2: Net-(Q66-Pad3) -> /FPGA and Power/RESET3
- R199 pad 1: /Rope Drivers/BPLIZ2 -> Net-(D95-Pad1)
- R199 pad 2: Net-(D96-Pad1) -> Net-(Q66-Pad3)
- R200 pad 1: Net-(D97-Pad2) -> /Rope Drivers/BPLIZ1
- R200 pad 2: GND -> Net-(D95-Pad1)
- R201 pad 1: /Rope Drivers/BPLIZ2 -> Net-(D96-Pad2)
- R201 pad 2: Net-(Q67-Pad2) -> GND
- R202 pad 1: Net-(Q68-Pad2) -> /Rope Drivers/BPLIZ1
- R202 pad 2: Net-(R202-Pad2) -> Net-(Q67-Pad2)
- R203 pad 1: Net-(R202-Pad2) -> Net-(Q68-Pad2)
- R203 pad 2: Net-(L19-Pad1) -> Net-(R203-Pad2)
- R204 pad 1: Net-(Q69-Pad2) -> Net-(R203-Pad2)
- R204 pad 2: Net-(R204-Pad2) -> Net-(L19-Pad1)
- R205 pad 1: Net-(R204-Pad2) -> Net-(Q69-Pad2)
- R205 pad 2: Net-(L20-Pad1) -> Net-(R205-Pad2)
- R206 pad 1: Net-(Q70-Pad1) -> Net-(R205-Pad2)
- R206 pad 2: /FPGA and Power/RESET3 -> Net-(L20-Pad1)
- R207 pad 1: Net-(D103-Pad1) -> Net-(Q70-Pad1)
- R207 pad 2: Net-(Q70-Pad3) -> /FPGA and Power/RESET2
- R208 pad 1: /Rope Drivers/BPLIZ1 -> Net-(D102-Pad1)
- R208 pad 2: Net-(D103-Pad1) -> Net-(Q70-Pad3)
- R209 pad 1: Net-(D104-Pad2) -> /Rope Drivers/BPLIZ2
- R209 pad 2: GND -> Net-(D102-Pad1)
- R210 pad 1: /Rope Drivers/BPLIZ1 -> Net-(D103-Pad2)
- R210 pad 2: Net-(Q71-Pad2) -> GND
- R211 pad 1: Net-(Q72-Pad2) -> /Rope Drivers/BPLIZ2
- R211 pad 2: Net-(R211-Pad2) -> Net-(Q71-Pad2)
- R212 pad 1: Net-(R211-Pad2) -> Net-(Q72-Pad2)
- R212 pad 2: Net-(L21-Pad1) -> Net-(R212-Pad2)
- R213 pad 1: Net-(Q73-Pad2) -> Net-(R212-Pad2)
- R213 pad 2: Net-(R213-Pad2) -> Net-(L21-Pad1)
- R214 pad 1: Net-(R213-Pad2) -> Net-(Q73-Pad2)
- R214 pad 2: Net-(L22-Pad1) -> Net-(R214-Pad2)
- R215 pad 1: Net-(Q74-Pad1) -> Net-(R214-Pad2)
- R215 pad 2: /FPGA and Power/RESET2 -> Net-(L22-Pad1)
- R216 pad 1: Net-(D110-Pad1) -> Net-(Q74-Pad1)
- R216 pad 2: Net-(Q74-Pad3) -> /FPGA and Power/RESET1
- R217 pad 1: /Rope Drivers/BPLIZ2 -> Net-(D109-Pad1)
- R217 pad 2: Net-(D110-Pad1) -> Net-(Q74-Pad3)
- R218 pad 1: Net-(D111-Pad2) -> /Rope Drivers/BPLIZ1
- R218 pad 2: GND -> Net-(D109-Pad1)
- R219 pad 1: /Rope Drivers/BPLIZ2 -> Net-(D110-Pad2)
- R219 pad 2: Net-(Q75-Pad2) -> GND
- R220 pad 1: Net-(Q76-Pad2) -> /Rope Drivers/BPLIZ1
- R220 pad 2: Net-(R220-Pad2) -> Net-(Q75-Pad2)
- R221 pad 1: Net-(R220-Pad2) -> Net-(Q76-Pad2)
- R221 pad 2: Net-(L23-Pad1) -> Net-(R221-Pad2)
- R222 pad 1: Net-(Q77-Pad2) -> Net-(R221-Pad2)
- R222 pad 2: Net-(R222-Pad2) -> Net-(L23-Pad1)
- R223 pad 1: Net-(R222-Pad2) -> Net-(Q77-Pad2)
- R223 pad 2: Net-(L24-Pad1) -> Net-(R223-Pad2)
- R224 pad 1: Net-(Q78-Pad1) -> Net-(R223-Pad2)
- R224 pad 2: /FPGA and Power/RESET1 -> Net-(L24-Pad1)
- R225 pad 1: Net-(D117-Pad1) -> Net-(Q78-Pad1)
- R225 pad 2: Net-(Q78-Pad3) -> /FPGA and Power/SET2
- R226 pad 1: /Rope Drivers/BPLIZ1 -> Net-(D116-Pad1)
- R226 pad 2: Net-(D117-Pad1) -> Net-(Q78-Pad3)
- R227 pad 1: Net-(D118-Pad2) -> /Rope Drivers/BPLIZ2
- R227 pad 2: GND -> Net-(D116-Pad1)
- R228 pad 1: /Rope Drivers/BPLIZ1 -> Net-(D117-Pad2)
- R228 pad 2: Net-(Q79-Pad2) -> GND
- R229 pad 1: Net-(Q80-Pad2) -> /Rope Drivers/BPLIZ2
- R229 pad 2: Net-(R229-Pad2) -> Net-(Q79-Pad2)
- R230 pad 1: Net-(R229-Pad2) -> Net-(Q80-Pad2)
- R230 pad 2: Net-(L25-Pad1) -> Net-(R230-Pad2)
- R231 pad 1: Net-(Q81-Pad2) -> Net-(R230-Pad2)
- R231 pad 2: Net-(R231-Pad2) -> Net-(L25-Pad1)
- R232 pad 1: Net-(R231-Pad2) -> Net-(Q81-Pad2)
- R232 pad 2: Net-(L26-Pad1) -> Net-(R232-Pad2)
- R233 pad 1: Net-(Q82-Pad1) -> Net-(R232-Pad2)
- R233 pad 2: /FPGA and Power/SET2 -> Net-(L26-Pad1)
- R234 pad 1: Net-(D124-Pad1) -> Net-(Q82-Pad1)
- R234 pad 2: Net-(Q82-Pad3) -> /FPGA and Power/SET1
- R235 pad 1: /Rope Drivers/BPLIZ2 -> Net-(D123-Pad1)
- R235 pad 2: Net-(D124-Pad1) -> Net-(Q82-Pad3)
- R236 pad 1: Net-(D125-Pad2) -> /Rope Drivers/BPLIZ1
- R236 pad 2: GND -> Net-(D123-Pad1)
- R237 pad 1: /Rope Drivers/BPLIZ2 -> Net-(D124-Pad2)
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Routing:
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
Commit message: Driver: updated to KiCad 6.0
Connections:
- net /FPGA and Power/~IL1 renamed /FPGA and Power/~{IL1}
- net /FPGA and Power/~IL2 renamed /FPGA and Power/~{IL2}
- net /FPGA and Power/~IL3 renamed /FPGA and Power/~{IL3}
- net /FPGA and Power/~IL4 renamed /FPGA and Power/~{IL4}
- net /FPGA and Power/~IL5 renamed /FPGA and Power/~{IL5}
- net /FPGA and Power/~IL6 renamed /FPGA and Power/~{IL6}
- net /FPGA and Power/~IL7 renamed /FPGA and Power/~{IL7}
- net /FPGA and Power/~IL8 renamed /FPGA and Power/~{IL8}
Other:
- net class Default removed

Commit message: Driver: incorporated most changes from the test board, and began layout
Parts:
- removed J5: DIN41612_03x32_C, Connector_DIN:DIN41612_C_3x32_Male_Horizontal_THT
- added C1: 1.0uF, Capacitor_Tantalum_SMD:CP_EIA-3528-21_Kemet-B, F.Cu at (404.1, 131.7)
- added C2: 1.0uF, Capacitor_Tantalum_SMD:CP_EIA-3528-21_Kemet-B, F.Cu at (717.3, -168.9)
- added C56: 0.1uF, Capacitor_SMD:C_0603_1608Metric, F.Cu at (416.3, -98.9)
- added C57: 0.1uF, Capacitor_SMD:C_0603_1608Metric, F.Cu at (412.3, -98.9)
- added C58: 4.7uF, Capacitor_SMD:C_0805_2012Metric, F.Cu at (403.3, 330.6)
- added C59: 1.0uF, Capacitor_SMD:C_0603_1608Metric, F.Cu at (408.0, 325.9)
- added D160: 1N4148, lachesis:D_SOD-323, F.Cu at (408.3, 353.2)
- added D161: 1N4148, lachesis:D_SOD-323, F.Cu at (413.2, 348.8)
- added D162: 1N4148, lachesis:D_SOD-323, F.Cu at (403.4, 360.6)
- added F1: 250mA, Fuse:Fuse_0603_1608Metric, F.Cu at (1001.3, 155.4)
- added F10: 250mA, Fuse:Fuse_0603_1608Metric, F.Cu at (511.0, 285.5)
- added F2: 250mA, Fuse:Fuse_0603_1608Metric, F.Cu at (413.0, 195.8)
- added F3: 250mA, Fuse:Fuse_0603_1608Metric, F.Cu at (726.1, -104.8)
- added F4: 250mA, Fuse:Fuse_0603_1608Metric, F.Cu at (609.1, -39.8)
- added F5: 250mA, Fuse:Fuse_0603_1608Metric, F.Cu at (511.0, 90.3)
- added F6: 250mA, Fuse:Fuse_0603_1608Metric, F.Cu at (1099.3, 25.3)
- added F7: 250mA, Fuse:Fuse_0603_1608Metric, F.Cu at (511.0, 25.3)
- added F8: 250mA, Fuse:Fuse_0603_1608Metric, F.Cu at (1197.4, -39.8)
- added F9: 250mA, Fuse:Fuse_0603_1608Metric, F.Cu at (628.1, -104.8)
- added H1: MountingHole_Pad, lachesis:MountingHole_No2_Pad, F.Cu at (58.2, 28.3)
- added H2: MountingHole_Pad, lachesis:MountingHole_No2_Pad, F.Cu at (107.7, 28.3)
- added H3: MountingHole_Pad, lachesis:MountingHole_No2_Pad, F.Cu at (157.2, 28.3)
- added H4: MountingHole_Pad, lachesis:MountingHole_No2_Pad, F.Cu at (228.6, 28.3)
- added H5: MountingHole_Pad, lachesis:MountingHole_No2_Pad, F.Cu at (58.2, 133.3)
- added H6: MountingHole_Pad, lachesis:MountingHole_No2_Pad, F.Cu at (107.7, 133.3)
- added H7: MountingHole_Pad, lachesis:MountingHole_No2_Pad, F.Cu at (157.2, 133.3)
- added H8: MountingHole_Pad, lachesis:MountingHole_No2_Pad, F.Cu at (228.6, 133.3)
- added JP1: Jumper_2_Open, Connector_PinHeader_2.00mm:PinHeader_1x02_P2.00mm_Vertical, F.Cu at (818.4, -169.1)
- added JP2: Jumper_2_Open, Connector_PinHeader_2.00mm:PinHeader_1x02_P2.00mm_Vertical, F.Cu at (814.3, -163.0)
- added JP3: Jumper_2_Open, Connector_PinHeader_2.00mm:PinHeader_1x02_P2.00mm_Vertical, F.Cu at (814.3, -169.1)
- added JP4: Jumper_2_Open, Connector_PinHeader_2.00mm:PinHeader_1x02_P2.00mm_Vertical, F.Cu at (1112.5, -104.0)
- added JP5: Jumper_2_Open, Connector_PinHeader_2.00mm:PinHeader_1x02_P2.00mm_Vertical, F.Cu at (1108.5, -98.0)
- added JP6: Jumper_2_Open, Connector_PinHeader_2.00mm:PinHeader_1x02_P2.00mm_Vertical, F.Cu at (1108.5, -104.0)
- added R268: 1k, Resistor_SMD:R_0603_1608Metric, F.Cu at (421.5, 348.6)
- added R269: 5.1k, Resistor_SMD:R_0603_1608Metric, F.Cu at (417.5, 348.6)
- added R270: 5.1k, Resistor_SMD:R_0603_1608Metric, F.Cu at (412.9, 351.5)
- added R271: 680, Resistor_SMD:R_0603_1608Metric, F.Cu at (403.1, 363.4)
- added R272: 5.1k, Resistor_SMD:R_0603_1608Metric, F.Cu at (407.7, 360.4)
- added R273: 3k, Resistor_SMD:R_0603_1608Metric, F.Cu at (417.5, 351.1)
- added R274: 10, Resistor_SMD:R_0603_1608Metric, F.Cu at (412.6, 354.0)
- added R275: NOM, Resistor_SMD:R_0603_1608Metric, F.Cu at (412.4, 356.5)
- added U19: AD1582BRTZ, Package_TO_SOT_SMD:SOT-23, F.Cu at (403.5, 326.9)
- C10, C11, C6, C7: value 0.1uF -> 6.8uF; footprint Capacitor_SMD:C_0603_1608Metric -> Capacitor_Tantalum_SMD:CP_EIA-7343-31_Kemet-D
- C12, C4, C8: value 10nF -> 6.8uF; footprint Capacitor_SMD:C_0603_1608Metric -> Capacitor_Tantalum_SMD:CP_EIA-7343-31_Kemet-D
- C13, C17, C21, C25, C29, C33: value 100pF -> 0.01uF
- C14, C18, C22, C26, C30, C34, C51: value 0.1uF -> 100pF
- C15, C19, C23, C27, C31, C35, C52: value 0.1uF -> 0.01uF
- C16, C20, C24, C28, C32: value 10nF -> 0.01uF
- C36, C37, C39, C40, C41, C43, C44: value 6.8uF -> 0.01uF; footprint Capacitor_Tantalum_SMD:CP_EIA-7343-31_Kemet-D -> Capacitor_SMD:C_0603_1608Metric
- C38, C42: value 6.8uF -> 100pF; footprint Capacitor_Tantalum_SMD:CP_EIA-7343-31_Kemet-D -> Capacitor_SMD:C_0603_1608Metric
- C45, C46: value 1.0uF -> 0.1uF; footprint Capacitor_Tantalum_SMD:CP_EIA-3216-18_Kemet-A -> Capacitor_SMD:C_0603_1608Metric
- C47, C48: value 0.1uF -> 1.0uF; footprint Capacitor_SMD:C_0603_1608Metric -> Capacitor_SMD:C_0805_2012Metric
- C49: value 0.33uF -> 1.0uF
- C5, C9: value 100pF -> 6.8uF; footprint Capacitor_SMD:C_0603_1608Metric -> Capacitor_Tantalum_SMD:CP_EIA-7343-31_Kemet-D
- C50: value 10nF -> 1.0uF
- D1, D10, D100, D101, D102, D103, D104, D105, D106, D107, D108, D109, D11, D110, D111, D112, D113, D114, D115, D116, D117, D118, D119, D12, D120, D121, D122, D123, D124, D125, D126, D127, D128, D129, D13, D130, D131, D132, D133, D134, D135, D136, D137, D138, D139, D14, D140, D141, D142, D143, D144, D145, D146, D147, D148, D149, D15, D150, D151, D152, D153, D154, D158, D159, D16, D17, D18, D19, D2, D20, D21, D22, D23, D24, D25, D26, D27, D28, D29, D3, D30, D31, D32, D33, D34, D35, D36, D37, D38, D39, D4, D40, D41, D42, D43, D44, D45, D46, D47, D48, D49, D5, D50, D51, D52, D53, D54, D55, D56, D57, D58, D59, D6, D60, D61, D62, D63, D64, D65, D66, D67, D68, D69, D7, D70, D71, D72, D73, D74, D75, D76, D77, D78, D79, D8, D80, D81, D82, D83, D84, D85, D86, D87, D88, D89, D9, D90, D91, D92, D93, D94, D95, D96, D97, D98, D99: footprint Diode_SMD:D_SOD-323 -> lachesis:D_SOD-323
- D155: value 1N4148 -> BLUE; footprint Diode_SMD:D_SOD-323 -> LED_SMD:LED_0603_1608Metric
- D156: value 1N4148 -> TEAL; footprint Diode_SMD:D_SOD-323 -> LED_SMD:LED_0603_1608Metric
- D157: value 1N4148 -> ORANGE; footprint Diode_SMD:D_SOD-323 -> LED_SMD:LED_0603_1608Metric
- J1: value Barrel_Jack_Switch -> DIN41612_03x32_C; footprint Connector_BarrelJack:BarrelJack_Horizontal -> Connector_DIN:DIN41612_C_3x32_Male_Horizontal_THT
- J2: value Conn_01x24 -> Barrel_Jack_Switch; footprint Connector_PinSocket_2.54mm:PinSocket_1x24_P2.54mm_Vertical -> lachesis:BarrelJack_CUI_PJ-002A
- J3: value Conn_02x06_Top_Bottom -> Conn_01x24; footprint Connector_PinSocket_2.54mm:PinSocket_2x06_P2.54mm_Vertical -> Connector_PinSocket_2.54mm:PinSocket_1x24_P2.54mm_Vertical
- L1, L2: value 8.2uH -> 2.2uH; footprint Inductor_SMD:L_1812_4532Metric -> lachesis:API_Delevan_1812R
- L10, L11, L12, L13, L14, L15, L16, L17, L18, L19, L20, L21, L22, L23, L24, L25, L26, L27, L28, L29, L3, L30, L31, L32, L33, L34, L35, L36, L4, L5, L6, L7, L8, L9: footprint Inductor_SMD:L_1812_4532Metric -> lachesis:API_Delevan_1812R
- L37, L38: value 2.2uH -> 8.2uH; footprint Inductor_SMD:L_1812_4532Metric -> lachesis:API_Delevan_1812R
- Q11, Q13, Q15, Q17, Q19, Q2, Q21, Q23, Q25, Q27, Q5, Q57, Q63, Q67, Q7, Q71, Q75, Q79, Q83, Q9: value MMBT2907 -> MMBT2222
- Q34, Q37, Q40, Q44, Q48, Q52, Q56, Q64, Q66, Q68, Q70, Q72, Q74, Q76, Q78, Q80, Q82, Q84, Q86, Q89: value MMBT2222 -> MMBT2907
- Q87: value MMBT2222 -> IRF7413; footprint Package_TO_SOT_SMD:SOT-23 -> Package_SO:SO-8_3.9x4.9mm_P1.27mm
- Q90: value IRF7413 -> MMBT2222; footprint Package_SO:SO-8_3.9x4.9mm_P1.27mm -> Package_TO_SOT_SMD:SOT-23
- R1: value 1.27k -> 1k
- R10, R18, R26, R34, R42, R50, R58: value 470 -> 390
- R100, R108, R120: value 5.1k -> 1k
- R101, R121, R93: value 2k -> 5.1k
- R102, R110, R122: value 3k -> 5.1k
- R103, R123: value 1k -> 27
- R104, R88: value 5.1k -> 7.5; footprint Resistor_SMD:R_0603_1608Metric -> Resistor_SMD:R_0805_2012Metric
- R105, R89: value 2k -> NOM
- R106, R86: value 3k -> 7.5; footprint Resistor_SMD:R_0603_1608Metric -> Resistor_SMD:R_0805_2012Metric
- R107, R127, R87: value 1k -> NOM
- R109, R181, R81: value 2k -> 1k
- R11, R19, R27, R3, R35, R43, R51, R59: value 2.7k -> 4.7
- R111, R131, R83: value 1k -> 5.1k
- R112: value 5.1k -> 27
- R113, R97: value 2k -> 7.5; footprint Resistor_SMD:R_0603_1608Metric -> Resistor_SMD:R_0805_2012Metric
- R114, R98: value 3k -> NOM
- R115, R135, R95: value 1k -> 7.5; footprint Resistor_SMD:R_0603_1608Metric -> Resistor_SMD:R_0805_2012Metric
- R116, R96: value 5.1k -> NOM
- R117: value 2k -> 3k
- R12, R20, R28, R36, R4, R44, R52, R60: value 2.7k -> NOM
- R124: value 390 -> 7.5; footprint Resistor_SMD:R_0603_1608Metric -> Resistor_SMD:R_0805_2012Metric
- R125: value 3.9 -> NOM
- R126: value NOM -> 7.5; footprint Resistor_SMD:R_0603_1608Metric -> Resistor_SMD:R_0805_2012Metric
- R128: value 390 -> 1k
- R129, R137, R141, R145, R149, R153, R157, R161, R165, R169, R173, R177: value 3.9 -> 1k
- R13, R21, R29, R37, R45, R5, R53, R61: value 2.7k -> 1k
- R130, R138, R142, R146, R150, R154, R158, R162, R166, R170, R174, R178: value NOM -> 5.1k
- R132: value 390 -> 27
- R133: value 3.9 -> 7.5; footprint Resistor_SMD:R_0603_1608Metric -> Resistor_SMD:R_0805_2012Metric
- R136: value 390 -> NOM
- R139, R143, R147, R151, R155, R159, R163, R167, R171, R175, R179, R251, R67: value 1k -> 2k
- R14, R22, R30, R38, R46, R54, R6, R62: value 2.7k -> 390
- R140, R144, R148, R152, R156, R160, R164, R168, R172, R176: value 390 -> 3k
- R15, R23, R39, R47, R55, R7: value 470 -> 4.7
- R16, R24, R32, R40, R48, R56, R64, R8: value 470 -> NOM
- R17, R25, R33, R41, R49, R57, R65, R9: value 470 -> 1k
- R180: value 470 -> 3k
- R182: value 750 -> 5.1k
- R184: value 1k -> 3k
- R185: value 470 -> 2.7k
- R186, R188: value 2k -> 2.7k
- R187: value 750 -> 2.7k
- R189, R190, R198, R199, R207, R208, R216: value 1k -> 100
- R191, R192, R200, R237: value 5.1k -> 100
- R193, R202, R211, R220: value 27 -> 2.7k
- R194, R196, R203, R212, R241: value 7.5 -> 2.7k
- R195, R204, R233, R242: value NOM -> 2.7k
- R197, R206, R213, R215, R222, R224, R231, R240: value NOM -> 100
- R2: value 249 -> 390
- R201, R209, R210, R218, R219, R227, R228, R236: value 5.1k -> 2.7k
- R205, R214, R221, R223, R230, R232, R239: value 7.5 -> 100
- R217, R225, R226, R234, R235: value 1k -> 2.7k
- R229, R238: value 27 -> 100
- R243, R244: value 200 -> 2.7k
- R245, R246, R247, R248: value 200 -> 100
- R249, R250: value 3k -> 0; footprint Resistor_SMD:R_0603_1608Metric -> Resistor_SMD:R_0805_2012Metric
- R252: value 390 -> 2k
- R253: value 2.2 -> 12k
- R254: value NOM -> 2.4k
- R255: value 1k -> 1020k
- R256: value 390 -> 2.87k
- R257: value 2.2 -> 9.76k
- R258: value NOM -> 54.9k
- R259: value 1020k -> 0.025; footprint Resistor_SMD:R_0603_1608Metric -> Resistor_SMD:R_1206_3216Metric
- R260: value 2.87k -> 10
- R261: value 9.76k -> 1k
- R262: value 54.9k -> 10k
- R263: value 0.025 -> 10k
- R264: value 10 -> 2.5k
- R266: value 10k -> 1.27k
- R267: value 10k -> 249
- R31, R63: value 470 -> 2.2
- R68: value 5.1k -> 750
- R69: value 5.1k -> 2k
- R70: value 680 -> 1k
- R71: value 5.1k -> 470
- R72: value 3k -> 2k
- R73: value 8.2 -> 750
- R74: value NOM -> 2k
- R75, R79: value 1k -> 200
- R76, R80: value 5.1k -> 200
- R77: value 2k -> 200
- R78: value 3k -> 200
- R82, R90: value 3k -> 1k
- R85: value 2k -> 27
- R94: value 3k -> 27
- U1: value AD1582BRTZ -> SN7524; footprint Package_TO_SOT_SMD:SOT-23 -> Package_DIP:DIP-16_W7.62mm_Socket
- U12: value JTE0624D05 -> ADP151-3.3; footprint Converter_DCDC:Converter_DCDC_XP_POWER_JTExxxxDxx_THT -> Package_TO_SOT_SMD:TSOT-23-5
- U9: value SN7524 -> JTE0624D05; footprint Package_DIP:DIP-16_W7.62mm_Socket -> Converter_DCDC:Converter_DCDC_XP_POWER_JTExxxxDxx_THT
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Connections:
- C10 pad 1: +5V -> /Rope Drivers/BPLIZ2
- C11 pad 1: GND -> /Sense Amplifiers/BPLSWX
- C11 pad 2: -5V -> GND
- C12 pad 1: GND -> /Strand Select/BPLSWZ
- C12 pad 2: /Sense Amplifiers/VREF -> GND
- C13 pad 2: Net-(C13-Pad2) -> /Sense Amplifiers/VREF
- C14 pad 1: +5V -> GND
- C14 pad 2: GND -> Net-(C14-Pad2)
- C15 pad 1: GND -> +5V
- C15 pad 2: -5V -> GND
- C16 pad 2: /Sense Amplifiers/VREF -> -5V
- C17 pad 2: Net-(C17-Pad2) -> /Sense Amplifiers/VREF
- C18 pad 1: +5V -> GND
- C18 pad 2: GND -> Net-(C18-Pad2)
- C19 pad 1: GND -> +5V
- C19 pad 2: -5V -> GND
- C20 pad 2: /Sense Amplifiers/VREF -> -5V
- C21 pad 2: Net-(C21-Pad2) -> /Sense Amplifiers/VREF
- C22 pad 1: +5V -> GND
- C22 pad 2: GND -> Net-(C22-Pad2)
- C23 pad 1: GND -> +5V
- C23 pad 2: -5V -> GND
- C24 pad 2: /Sense Amplifiers/VREF -> -5V
- C25 pad 2: Net-(C25-Pad2) -> /Sense Amplifiers/VREF
- C26 pad 1: +5V -> GND
- C26 pad 2: GND -> Net-(C26-Pad2)
- C27 pad 1: GND -> +5V
- C27 pad 2: -5V -> GND
- C28 pad 2: /Sense Amplifiers/VREF -> -5V
- C29 pad 2: Net-(C29-Pad2) -> /Sense Amplifiers/VREF
- C3 pad 1: /Sense Amplifiers/BPLSWX -> /Rope Drivers/BPLMX1
- C30 pad 1: +5V -> GND
- C30 pad 2: GND -> Net-(C30-Pad2)
- C31 pad 1: GND -> +5V
- C31 pad 2: -5V -> GND
- C32 pad 2: /Sense Amplifiers/VREF -> -5V
- C33 pad 2: Net-(C33-Pad2) -> /Sense Amplifiers/VREF
- C34 pad 1: +5V -> GND
- C34 pad 2: GND -> Net-(C34-Pad2)
- C35 pad 1: GND -> +5V
- C35 pad 2: -5V -> GND
- C36 pad 1: /Strand Select/BPLSWZ -> GND
- C36 pad 2: GND -> -5V
- C37 pad 1: /Rope Drivers/BPLIZ1 -> GND
- C37 pad 2: GND -> /Sense Amplifiers/VREF
- C38 pad 1: /Rope Drivers/BPLIZ2 -> GND
- C38 pad 2: GND -> Net-(C38-Pad2)
- C39 pad 1: /Rope Drivers/BPLMX1 -> +5V
- C4 pad 1: GND -> /Rope Drivers/BPLMX2
- C4 pad 2: /Sense Amplifiers/VREF -> GND
- C40 pad 1: /Rope Drivers/BPLMX2 -> GND
- C40 pad 2: GND -> -5V
- C41 pad 1: /Rope Drivers/BPLMX3 -> GND
- C41 pad 2: GND -> /Sense Amplifiers/VREF
- C42 pad 1: /Rope Drivers/BPLMX1 -> GND
- C42 pad 2: GND -> Net-(C42-Pad2)
- C43 pad 1: /Rope Drivers/BPLMX2 -> +5V
- C44 pad 1: /Rope Drivers/BPLMX3 -> GND
- C44 pad 2: GND -> -5V
- C45 pad 2: GND -> +3V3
- C46 pad 2: GND -> +3V3
- C47 pad 2: +3V3 -> -5V
- C48 pad 1: GND -> +5V
- C48 pad 2: +3V3 -> GND
- C49 pad 1: Net-(C49-Pad1) -> GND
- C49 pad 2: GND -> Net-(C49-Pad2)
- C5 pad 1: GND -> /Rope Drivers/BPLMY1
- C5 pad 2: Net-(C5-Pad2) -> GND
- C50 pad 1: Net-(C50-Pad1) -> +3V3
- C51 pad 1: GND -> Net-(C51-Pad1)
- C51 pad 2: +3V3 -> GND
- C52 pad 1: +3V3 -> Net-(C52-Pad1)
- C53 pad 1: +3V3 -> GND
- C53 pad 2: GND -> +3V3
- C6 pad 1: +5V -> /Rope Drivers/BPLMY2
- C7 pad 1: GND -> /Rope Drivers/BPLMX3
- C7 pad 2: -5V -> GND
- C8 pad 1: GND -> /Rope Drivers/BPLIZ1
- C8 pad 2: /Sense Amplifiers/VREF -> GND
- C9 pad 1: GND -> /Rope Drivers/BPLMY3
- C9 pad 2: Net-(C9-Pad2) -> GND
- D1 pad 1: GND -> Net-(D1-Pad1)
- D10 pad 1: GND -> Net-(D10-Pad1)
- D100 pad 1: Net-(D100-Pad1) -> GND
- D100 pad 2: /Rope Drivers/BPLIZ2 -> Net-(D100-Pad2)
- D101 pad 2: Net-(D100-Pad1) -> /Rope Drivers/BPLIZ2
- D103 pad 2: Net-(D103-Pad2) -> Net-(D102-Pad1)
- D104 pad 2: Net-(D103-Pad1) -> Net-(D104-Pad2)
- D106 pad 1: GND -> Net-(D106-Pad1)
- D107 pad 1: Net-(D107-Pad1) -> GND
- D107 pad 2: /Rope Drivers/BPLIZ1 -> Net-(D106-Pad1)
- D108 pad 2: Net-(D107-Pad1) -> /Rope Drivers/BPLIZ2
- D11 pad 2: /Strand Select/BPLSWZ -> Net-(D10-Pad1)
- D110 pad 2: Net-(D110-Pad2) -> Net-(D109-Pad1)
- D111 pad 2: Net-(D110-Pad1) -> Net-(D111-Pad2)
- D113 pad 1: GND -> Net-(D113-Pad1)
- D114 pad 1: Net-(D114-Pad1) -> GND
- D114 pad 2: /Rope Drivers/BPLIZ2 -> Net-(D113-Pad1)
- D115 pad 1: Net-(D115-Pad1) -> GND
- D115 pad 2: Net-(D114-Pad1) -> /Rope Drivers/40365A
- D116 pad 1: Net-(D116-Pad1) -> GND
- D116 pad 2: Net-(D115-Pad1) -> /Rope Drivers/40366A
- D117 pad 2: Net-(D117-Pad2) -> /Rope Drivers/BPLIZ1
- D12 pad 2: Net-(D12-Pad2) -> Net-(D11-Pad1)
- D120 pad 1: GND -> Net-(D120-Pad1)
- D120 pad 2: Net-(D119-Pad1) -> Net-(D120-Pad2)
- D121 pad 2: /Rope Drivers/BPLIZ1 -> Net-(D120-Pad1)
- D123 pad 1: Net-(D123-Pad1) -> GND
- D124 pad 2: Net-(D124-Pad2) -> /Rope Drivers/BPLIZ2
- D127 pad 1: GND -> Net-(D127-Pad1)
- D127 pad 2: Net-(D126-Pad1) -> Net-(D127-Pad2)
- D128 pad 1: /Connector/RFD1 -> Net-(D128-Pad1)
- D128 pad 2: /Rope Drivers/BPLMX1 -> Net-(D127-Pad1)
- D129 pad 1: /Connector/RFD3 -> Net-(D129-Pad1)
- D129 pad 2: /Rope Drivers/BPLMX2 -> Net-(D128-Pad1)
- D13 pad 2: /Strand Select/BPLSWZ -> Net-(D13-Pad2)
- D130 pad 1: /Connector/RSTRD4 -> GND
- D130 pad 2: /Rope Drivers/BPLMX3 -> Net-(D129-Pad1)
- D131 pad 1: /Connector/RCD1 -> GND
- D131 pad 2: /Rope Drivers/BPLMX1 -> Net-(D131-Pad2)
- D132 pad 1: /Connector/RCD3 -> Net-(D132-Pad1)
- D132 pad 2: /Rope Drivers/BPLMX2 -> /Strand Select/BPLSWZ
- D133 pad 1: /Connector/RFD2 -> GND
- D133 pad 2: /Rope Drivers/BPLMX1 -> Net-(D133-Pad2)
- D134 pad 1: /Connector/RFD4 -> Net-(D134-Pad1)
- D134 pad 2: /Rope Drivers/BPLMX2 -> /Strand Select/BPLSWZ
- D135 pad 1: /Connector/RSTRD3 -> GND
- D135 pad 2: /Rope Drivers/BPLMX3 -> Net-(D135-Pad2)
- D136 pad 1: /Connector/RCD2 -> Net-(D136-Pad1)
- D136 pad 2: /Rope Drivers/BPLMX1 -> /Strand Select/BPLSWZ
- D137 pad 1: /Connector/RCD4 -> GND
- D137 pad 2: /Rope Drivers/BPLMX2 -> Net-(D137-Pad2)
- D138 pad 1: /Connector/SETRN1 -> Net-(D138-Pad1)
- D138 pad 2: /Rope Drivers/BPLMX3 -> /Strand Select/BPLSWZ
- D139 pad 1: /Connector/RFD5 -> GND
- D139 pad 2: /Rope Drivers/BPLMX1 -> Net-(D139-Pad2)
- D14 pad 1: GND -> Net-(D14-Pad1)
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Routing:
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- added copper zone on F.Cu, net +14V
- added copper zone on F.Cu, net /FPGA and Power/14V_IN
- added copper zone on F.Cu, net /FPGA and Power/14V_SENSE
- added copper zone on In1.Cu, net GND
Other:
- board size 228.6 x 116.8 mm -> 228.6 x 110.7 mm
- copper layers 2 -> 6

Commit message: Driver: laid out most of the subcircuits
Parts:
- R31, R63: value 2.2 -> 4.7
- moved D76 1072.3 mm to (38.6, -25.3)
- moved D77 1072.3 mm to (38.6, -22.3)
- moved D78 1072.3 mm to (43.2, -25.4)
- moved D79 1072.3 mm to (38.6, -19.4)
- moved D80 1072.3 mm to (51.3, -37.4)
- moved D81 1072.3 mm to (47.3, -31.5)
- moved D82 1072.3 mm to (42.6, -28.4)
- moved D83 1072.3 mm to (42.6, -31.3)
- moved D85 1072.3 mm to (47.3, -34.4)
- moved JP4 1072.3 mm to (42.3, -36.8)
- moved JP5 1072.3 mm to (38.3, -30.8)
- moved JP6 1072.3 mm to (38.3, -36.8)
- moved R78 1072.3 mm to (47.0, -28.8)
- moved D84 1072.3 mm to (51.9, -34.4)
- moved D86 1072.3 mm to (46.7, -37.4)
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Connections:
- J1 pad c1: /Connector/GAR1 -> /Connector/GAR15
- J1 pad c10: /Connector/GAR10 -> /Connector/GBR4
- J1 pad c11: /Connector/GAR11 -> /Connector/GAR5
- J1 pad c12: /Connector/GAR12 -> /Connector/GBR5
- J1 pad c13: /Connector/GAR13 -> /Connector/GAR6
- J1 pad c14: /Connector/GAR14 -> /Connector/GBR6
- J1 pad c15: /Connector/GAR15 -> /Connector/GAR7
- J1 pad c16: /Connector/GAR16 -> /Connector/GBR7
- J1 pad c17: /Connector/GBR1 -> /Connector/GAR8
- J1 pad c18: /Connector/GBR2 -> /Connector/GBR8
- J1 pad c19: /Connector/GBR3 -> /Connector/GAR9
- J1 pad c2: /Connector/GAR2 -> /Connector/GBR15
- J1 pad c20: /Connector/GBR4 -> /Connector/GBR9
- J1 pad c21: /Connector/GBR5 -> /Connector/GAR10
- J1 pad c22: /Connector/GBR6 -> /Connector/GBR10
- J1 pad c23: /Connector/GBR7 -> /Connector/GAR11
- J1 pad c24: /Connector/GBR8 -> /Connector/GBR11
- J1 pad c25: /Connector/GBR9 -> /Connector/GAR12
- J1 pad c26: /Connector/GBR10 -> /Connector/GBR12
- J1 pad c27: /Connector/GBR11 -> /Connector/GAR13
- J1 pad c28: /Connector/GBR12 -> /Connector/GBR13
- J1 pad c29: /Connector/GBR13 -> /Connector/GAR14
- J1 pad c3: /Connector/GAR3 -> /Connector/GAR1
- J1 pad c31: /Connector/GBR15 -> /Connector/GAR16
- J1 pad c4: /Connector/GAR4 -> /Connector/GBR1
- J1 pad c5: /Connector/GAR5 -> /Connector/GAR2
- J1 pad c6: /Connector/GAR6 -> /Connector/GBR2
- J1 pad c7: /Connector/GAR7 -> /Connector/GAR3
- J1 pad c8: /Connector/GAR8 -> /Connector/GBR3
- J1 pad c9: /Connector/GAR9 -> /Connector/GAR4
- R187 pad 1: /Connector/GAR2 -> /Connector/GAR15
- R188 pad 2: /Connector/GBR2 -> /Connector/GBR15
- R195 pad 1: /Connector/GAR4 -> /Connector/GAR2
- R196 pad 2: /Connector/GBR4 -> /Connector/GBR2
- R203 pad 1: /Connector/GAR6 -> /Connector/GAR4
- R204 pad 2: /Connector/GBR6 -> /Connector/GBR4
- R211 pad 1: /Connector/GAR8 -> /Connector/GAR6
- R212 pad 2: /Connector/GBR8 -> /Connector/GBR6
- R219 pad 1: /Connector/GAR10 -> /Connector/GAR8
- R220 pad 2: /Connector/GBR10 -> /Connector/GBR8
- R227 pad 1: /Connector/GAR12 -> /Connector/GAR10
- R228 pad 2: /Connector/GBR12 -> /Connector/GBR10
- R235 pad 1: /Connector/GAR14 -> /Connector/GAR12
- R236 pad 2: /Connector/GBR14 -> /Connector/GBR12
- R241 pad 1: /Connector/GAR15 -> /Connector/GAR16
- R242 pad 2: /Connector/GBR15 -> /Connector/GBR16
- R243 pad 1: /Connector/GAR16 -> /Connector/GAR14
- R244 pad 2: /Connector/GBR16 -> /Connector/GBR14
- T10 pad 1: /Connector/GBR10 -> /Connector/GBR8
- T10 pad 3: /Connector/GAR10 -> /Connector/GAR8
- T12 pad 1: /Connector/GBR12 -> /Connector/GBR10
- T12 pad 3: /Connector/GAR12 -> /Connector/GAR10
- T14 pad 1: /Connector/GBR14 -> /Connector/GBR12
- T14 pad 3: /Connector/GAR14 -> /Connector/GAR12
- T15 pad 1: /Connector/GBR15 -> /Connector/GBR16
- T15 pad 3: /Connector/GAR15 -> /Connector/GAR16
- T16 pad 1: /Connector/GBR16 -> /Connector/GBR14
- T16 pad 3: /Connector/GAR16 -> /Connector/GAR14
- T2 pad 1: /Connector/GBR2 -> /Connector/GBR15
- T2 pad 3: /Connector/GAR2 -> /Connector/GAR15
- T4 pad 1: /Connector/GBR4 -> /Connector/GBR2
- T4 pad 3: /Connector/GAR4 -> /Connector/GAR2
- T6 pad 1: /Connector/GBR6 -> /Connector/GBR4
- T6 pad 3: /Connector/GAR6 -> /Connector/GAR4
- T8 pad 1: /Connector/GBR8 -> /Connector/GBR6
- T8 pad 3: /Connector/GAR8 -> /Connector/GAR6
Routing:
- net GND: track 6.78 -> 229.0 mm, vias 6 -> 106
- net /FPGA and Power/SBF: track 0.00 -> 89.1 mm
- net /Strand Select/BPLSWZ: track 0.00 -> 58.3 mm, vias 0 -> 13
- net /Rope Drivers/BPLIZ2: track 0.00 -> 47.1 mm, vias 0 -> 4
- net /Rope Drivers/BPLIZ1: track 0.00 -> 47.1 mm, vias 0 -> 4
- net /Sense Amplifiers/BPLSWX: track 0.00 -> 35.7 mm, vias 0 -> 16
- net /Sense Amplifiers/VREF: track 0.00 -> 32.2 mm
- net -5V: track 0.00 -> 26.9 mm
- net +5V: track 0.00 -> 26.9 mm
- net /Rope Drivers/40366A: track 0.00 -> 24.0 mm, vias 0 -> 13
- net /Rope Drivers/40365A: track 0.00 -> 24.0 mm, vias 0 -> 13
- net Net-(D120-Pad2): track 0.00 -> 15.4 mm
- net Net-(D111-Pad2): track 0.00 -> 15.4 mm
- net Net-(D104-Pad2): track 0.00 -> 15.4 mm
- net Net-(D90-Pad2): track 0.00 -> 15.4 mm
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