File: boards/driver/filtered_14v.kicad_sch (KiCad schematic)
At the start: 3 parts

Commit message: Driver: minor schematic cleanup and populated all of the BOM except for resistors
Parts:
- C11: MPN (none) -> T495D685K035ATE300; Manufacturer (none) -> KEMET; Package (none) -> 2917
- F9: MPN (none) -> 0467.250NR; Manufacturer (none) -> Littelfuse Inc; Package (none) -> 0603
- L37: MPN (none) -> 1812R-822J; Manufacturer (none) -> API Delevan Inc; Package (none) -> 1812
Changed lines of the file:
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@@
+      (effects (font (size 1.27 1.27)) hide)
+    )
+    (property "MPN" "0467.250NR" (id 4) (at 115.57 96.52 0)
+      (effects (font (size 1.27 1.27)) hide)
+    )
+    (property "Manufacturer" "Littelfuse Inc" (id 5) (at 115.57 96.52 0)
+      (effects (font (size 1.27 1.27)) hide)
+    )
+    (property "Description" "FUSE BOARD MOUNT 250MA 32VAC/VDC" (id 6) (at 115.57 96.52 0)
+      (effects (font (size 1.27 1.27)) hide)
+    )
+    (property "Package" "0603" (id 7) (at 115.57 96.52 0)
       (effects (font (size 1.27 1.27)) hide)
     )
@@
     )
     (property "Digikey" "https://www.digikey.com/en/products/detail/api-delevan-inc/1812R-822J/1115322" (id 8) (at 134.62 96.52 90)
+      (effects (font (size 1.27 1.27)) hide)
+    )
+    (property "MPN" "1812R-822J" (id 9) (at 134.62 96.52 0)
+      (effects (font (size 1.27 1.27)) hide)
+    )
+    (property "Manufacturer" "API Delevan Inc" (id 10) (at 134.62 96.52 0)
+      (effects (font (size 1.27 1.27)) hide)
+    )
+    (property "Description" "FIXED IND 8.2UH 375MA 1.4OHM SMD" (id 11) (at 134.62 96.52 0)
+      (effects (font (size 1.27 1.27)) hide)
+    )
+    (property "Package" "1812" (id 12) (at 134.62 96.52 0)
       (effects (font (size 1.27 1.27)) hide)
     )
@@
       (effects (font (size 1.27 1.27)) hide)
     )
+    (property "Description" "CAP TANT 6.8UF 10% 35V 2917" (id 9) (at 140.97 102.87 0)
+      (effects (font (size 1.27 1.27)) hide)
+    )
+    (property "MPN" "T495D685K035ATE300" (id 10) (at 140.97 102.87 0)
+      (effects (font (size 1.27 1.27)) hide)
+    )
+    (property "Manufacturer" "KEMET" (id 11) (at 140.97 102.87 0)
+      (effects (font (size 1.27 1.27)) hide)
+    )
+    (property "Package" "2917" (id 12) (at 140.97 102.87 0)
+      (effects (font (size 1.27 1.27)) hide)
+    )
