File: boards/driver/sense_amp_pair.kicad_sch (KiCad schematic)
At the start: 15 parts, among them T1 1:1, T2 1:1, U1 SN7524

Commit message: Driver: filled out the rest of the BOM, except for defaults for nominal resistances
Parts:
- R185, R186, R187, R188: MPN (none) -> ERJ-PB3B2701V; Manufacturer (none) -> Panasonic Electronic Components; Package (none) -> 0603; Rating (none) -> 1/5W; Tolerance (none) -> 0.1%
- R189, R190, R191, R192: MPN (none) -> ERA-3VEB1000V; Manufacturer (none) -> Panasonic Electronic Components; Package (none) -> 0603; Rating (none) -> 1/8W; Tolerance (none) -> 0.1%
Changed lines of the file:
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@@
+      (effects (font (size 1.27 1.27)) hide)
+    )
+    (property "Description" "RES SMD 2.7K PULSE-WITHSTANDING OHM 0.1% 1/5W 0603" (id 4) (at 73.66 46.99 0)
+      (effects (font (size 1.27 1.27)) hide)
+    )
+    (property "MPN" "ERJ-PB3B2701V" (id 5) (at 73.66 46.99 0)
+      (effects (font (size 1.27 1.27)) hide)
+    )
+    (property "Manufacturer" "Panasonic Electronic Components" (id 6) (at 73.66 46.99 0)
+      (effects (font (size 1.27 1.27)) hide)
+    )
+    (property "Package" "0603" (id 7) (at 73.66 46.99 0)
+      (effects (font (size 1.27 1.27)) hide)
+    )
+    (property "Rating" "1/5W" (id 8) (at 73.66 46.99 0)
+      (effects (font (size 1.27 1.27)) hide)
+    )
+    (property "Tolerance" "0.1%" (id 9) (at 73.66 46.99 0)
       (effects (font (size 1.27 1.27)) hide)
     )
@@
       (effects (font (size 1.27 1.27)) hide)
     )
+    (property "Description" "RES SMD 2.7K PULSE-WITHSTANDING OHM 0.1% 1/5W 0603" (id 4) (at 73.66 57.15 0)
+      (effects (font (size 1.27 1.27)) hide)
+    )
+    (property "MPN" "ERJ-PB3B2701V" (id 5) (at 73.66 57.15 0)
+      (effects (font (size 1.27 1.27)) hide)
+    )
+    (property "Manufacturer" "Panasonic Electronic Components" (id 6) (at 73.66 57.15 0)
+      (effects (font (size 1.27 1.27)) hide)
+    )
+    (property "Package" "0603" (id 7) (at 73.66 57.15 0)
+      (effects (font (size 1.27 1.27)) hide)
+    )
+    (property "Rating" "1/5W" (id 8) (at 73.66 57.15 0)
+      (effects (font (size 1.27 1.27)) hide)
+    )
+    (property "Tolerance" "0.1%" (id 9) (at 73.66 57.15 0)
+      (effects (font (size 1.27 1.27)) hide)
+    )
     (pin "1")
     (pin "2")
@@
       (effects (font (size 1.27 1.27)) hide)
     )
+    (property "Description" "RES 100 OHM 0.1% 1/8W 0603" (id 4) (at 111.76 46.99 0)
+      (effects (font (size 1.27 1.27)) hide)
+    )
+    (property "MPN" "ERA-3VEB1000V" (id 5) (at 111.76 46.99 0)
+      (effects (font (size 1.27 1.27)) hide)
+    )
+    (property "Manufacturer" "Panasonic Electronic Components" (id 6) (at 111.76 46.99 0)
+      (effects (font (size 1.27 1.27)) hide)
+    )
+    (property "Package" "0603" (id 7) (at 111.76 46.99 0)
+      (effects (font (size 1.27 1.27)) hide)
+    )
+    (property "Rating" "1/8W" (id 8) (at 111.76 46.99 0)
+      (effects (font (size 1.27 1.27)) hide)
+    )
+    (property "Tolerance" "0.1%" (id 9) (at 111.76 46.99 0)
+      (effects (font (size 1.27 1.27)) hide)
+    )
     (pin "1")
     (pin "2")
@@
     )
     (property "Datasheet" "~" (id 3) (at 111.76 57.15 0)
+      (effects (font (size 1.27 1.27)) hide)
+    )
+    (property "Description" "RES 100 OHM 0.1% 1/8W 0603" (id 4) (at 111.76 57.15 0)
+      (effects (font (size 1.27 1.27)) hide)
+    )
+    (property "MPN" "ERA-3VEB1000V" (id 5) (at 111.76 57.15 0)
+      (effects (font (size 1.27 1.27)) hide)
+    )
+    (property "Manufacturer" "Panasonic Electronic Components" (id 6) (at 111.76 57.15 0)
+      (effects (font (size 1.27 1.27)) hide)
+    )
+    (property "Package" "0603" (id 7) (at 111.76 57.15 0)
+      (effects (font (size 1.27 1.27)) hide)
+    )
+    (property "Rating" "1/8W" (id 8) (at 111.76 57.15 0)
+      (effects (font (size 1.27 1.27)) hide)
+    )
+    (property "Tolerance" "0.1%" (id 9) (at 111.76 57.15 0)
       (effects (font (size 1.27 1.27)) hide)
     )
@@
       (effects (font (size 1.27 1.27)) hide)
     )
+    (property "Description" "RES SMD 2.7K PULSE-WITHSTANDING OHM 0.1% 1/5W 0603" (id 4) (at 73.66 72.39 0)
+      (effects (font (size 1.27 1.27)) hide)
+    )
+    (property "MPN" "ERJ-PB3B2701V" (id 5) (at 73.66 72.39 0)
+      (effects (font (size 1.27 1.27)) hide)
+    )
+    (property "Manufacturer" "Panasonic Electronic Components" (id 6) (at 73.66 72.39 0)
+      (effects (font (size 1.27 1.27)) hide)
+    )
+    (property "Package" "0603" (id 7) (at 73.66 72.39 0)
+      (effects (font (size 1.27 1.27)) hide)
+    )
+    (property "Rating" "1/5W" (id 8) (at 73.66 72.39 0)
+      (effects (font (size 1.27 1.27)) hide)
+    )
+    (property "Tolerance" "0.1%" (id 9) (at 73.66 72.39 0)
+      (effects (font (size 1.27 1.27)) hide)
+    )
     (pin "1")
     (pin "2")
@@
       (effects (font (size 1.27 1.27)) hide)
     )
+    (property "Description" "RES SMD 2.7K PULSE-WITHSTANDING OHM 0.1% 1/5W 0603" (id 4) (at 73.66 82.55 0)
+      (effects (font (size 1.27 1.27)) hide)
+    )
+    (property "MPN" "ERJ-PB3B2701V" (id 5) (at 73.66 82.55 0)
+      (effects (font (size 1.27 1.27)) hide)
+    )
+    (property "Manufacturer" "Panasonic Electronic Components" (id 6) (at 73.66 82.55 0)
+      (effects (font (size 1.27 1.27)) hide)
+    )
+    (property "Package" "0603" (id 7) (at 73.66 82.55 0)
+      (effects (font (size 1.27 1.27)) hide)
+    )
+    (property "Rating" "1/5W" (id 8) (at 73.66 82.55 0)
+      (effects (font (size 1.27 1.27)) hide)
+    )
+    (property "Tolerance" "0.1%" (id 9) (at 73.66 82.55 0)
+      (effects (font (size 1.27 1.27)) hide)
+    )
     (pin "1")
     (pin "2")
@@
       (effects (font (size 1.27 1.27)) hide)
     )
+    (property "Description" "RES 100 OHM 0.1% 1/8W 0603" (id 4) (at 111.76 72.39 0)
+      (effects (font (size 1.27 1.27)) hide)
+    )
+    (property "MPN" "ERA-3VEB1000V" (id 5) (at 111.76 72.39 0)
+      (effects (font (size 1.27 1.27)) hide)
+    )
+    (property "Manufacturer" "Panasonic Electronic Components" (id 6) (at 111.76 72.39 0)
+      (effects (font (size 1.27 1.27)) hide)
+    )
+    (property "Package" "0603" (id 7) (at 111.76 72.39 0)
+      (effects (font (size 1.27 1.27)) hide)
+    )
+    (property "Rating" "1/8W" (id 8) (at 111.76 72.39 0)
+      (effects (font (size 1.27 1.27)) hide)
+    )
+    (property "Tolerance" "0.1%" (id 9) (at 111.76 72.39 0)
+      (effects (font (size 1.27 1.27)) hide)
+    )
     (pin "1")
     (pin "2")
@@
       (effects (font (size 1.27 1.27)) hide)
     )
+    (property "Description" "RES 100 OHM 0.1% 1/8W 0603" (id 4) (at 111.76 82.55 0)
+      (effects (font (size 1.27 1.27)) hide)
+    )
+    (property "MPN" "ERA-3VEB1000V" (id 5) (at 111.76 82.55 0)
+      (effects (font (size 1.27 1.27)) hide)
+    )
+    (property "Manufacturer" "Panasonic Electronic Components" (id 6) (at 111.76 82.55 0)
+      (effects (font (size 1.27 1.27)) hide)
+    )
+    (property "Package" "0603" (id 7) (at 111.76 82.55 0)
+      (effects (font (size 1.27 1.27)) hide)
+    )
+    (property "Rating" "1/8W" (id 8) (at 111.76 82.55 0)
+      (effects (font (size 1.27 1.27)) hide)
+    )
+    (property "Tolerance" "0.1%" (id 9) (at 111.76 82.55 0)
+      (effects (font (size 1.27 1.27)) hide)
+    )
