File: boards/driver_test/ihenv.kicad_sch (KiCad schematic)
At the start: 8 parts, among them Q15 MMBT2222, Q16 MMBT2907, Q17 MMBT2222

Commit message: Driver: some high-level board rearrangement and addition of 3d models
Connections:
- net 0V renamed 4036nA
- net PWR renamed BPLIZ
Changed lines of the file:
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@@
     (stroke (width 0) (type default) (color 0 0 0 0))
   )
-  (hierarchical_label "0V" (shape input) (at 90.17 102.87 180)
+  (hierarchical_label "4036nA" (shape input) (at 90.17 102.87 180)
     (effects (font (size 1.27 1.27)) (justify right))
   )
@@
     (effects (font (size 1.27 1.27)) (justify right))
   )
-  (hierarchical_label "PWR" (shape input) (at 99.06 66.04 180)
+  (hierarchical_label "BPLIZ" (shape input) (at 99.06 66.04 180)
     (effects (font (size 1.27 1.27)) (justify right))
   )

Commit message: Driver test: finished up board layout
Parts:
- renumbered R56 to R58, R57 to R59, R58 to R60, R59 to R61, R60 to R62
Changed lines of the file:
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@@
   (symbol (lib_id "Device:R_US") (at 100.33 92.71 270) (unit 1)
     (in_bom yes) (on_board yes)
-    (property "Reference" "R56" (id 0) (at 100.33 87.503 90))
+    (property "Reference" "R58" (id 0) (at 100.33 87.503 90))
     (property "Value" "1k" (id 1) (at 100.33 89.8144 90))
     (property "Footprint" "Resistor_SMD:R_0603_1608Metric" (id 2) (at 100.076 93.726 90)
@@
   (symbol (lib_id "power:GND") (at 143.51 106.68 0) (unit 1)
     (in_bom yes) (on_board yes)
-    (property "Reference" "#PWR051" (id 0) (at 143.51 113.03 0)
+    (property "Reference" "#PWR055" (id 0) (at 143.51 113.03 0)
       (effects (font (size 1.27 1.27)) hide)
     )
@@
   (symbol (lib_id "Device:R_US") (at 114.3 82.55 0) (unit 1)
     (in_bom yes) (on_board yes)
-    (property "Reference" "R58" (id 0) (at 116.0272 81.3816 0)
+    (property "Reference" "R60" (id 0) (at 116.0272 81.3816 0)
       (effects (font (size 1.27 1.27)) (justify left))
     )
@@
   (symbol (lib_id "Device:R_US") (at 114.3 72.39 0) (unit 1)
     (in_bom yes) (on_board yes)
-    (property "Reference" "R57" (id 0) (at 116.0272 71.2216 0)
+    (property "Reference" "R59" (id 0) (at 116.0272 71.2216 0)
       (effects (font (size 1.27 1.27)) (justify left))
     )
@@
   (symbol (lib_id "Device:R_US") (at 129.54 93.98 0) (unit 1)
     (in_bom yes) (on_board yes)
-    (property "Reference" "R59" (id 0) (at 131.2672 92.8116 0)
+    (property "Reference" "R61" (id 0) (at 131.2672 92.8116 0)
       (effects (font (size 1.27 1.27)) (justify left))
     )
@@
   (symbol (lib_id "Device:R_US") (at 143.51 99.06 0) (unit 1)
     (in_bom yes) (on_board yes)
-    (property "Reference" "R60" (id 0) (at 145.2372 97.8916 0)
+    (property "Reference" "R62" (id 0) (at 145.2372 97.8916 0)
       (effects (font (size 1.27 1.27)) (justify left))
     )
