File: boards/driver_test/inhibit.kicad_sch (KiCad schematic)
At the start: 11 parts, among them Q22 MMBT2222, Q23 MMBT2222

Commit message: Driver: some high-level board rearrangement and addition of 3d models
Connections:
- net 0V renamed 4036nA
- net PWR renamed 4033nA
Changed lines of the file:
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@@
     (effects (font (size 1.27 1.27)) (justify right))
   )
-  (hierarchical_label "0V" (shape input) (at 74.93 100.33 180)
+  (hierarchical_label "4036nA" (shape input) (at 74.93 100.33 180)
     (effects (font (size 1.27 1.27)) (justify right))
   )
-  (hierarchical_label "PWR" (shape input) (at 91.44 63.5 180)
+  (hierarchical_label "4033nA" (shape input) (at 91.44 63.5 180)
     (effects (font (size 1.27 1.27)) (justify right))
   )

Commit message: Driver test: finished up board layout
Parts:
- renumbered R69 to R71, R70 to R72, R71 to R73, R72 to R74
Changed lines of the file:
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@@
   (symbol (lib_id "Device:R_US") (at 92.71 90.17 270)
     (in_bom yes) (on_board yes)
-    (property "Reference" "R69" (id 0) (at 92.71 84.963 90))
+    (property "Reference" "R71" (id 0) (at 92.71 84.963 90))
     (property "Value" "1k" (id 1) (at 92.71 87.2744 90))
     (property "Footprint" "Resistor_SMD:R_0603_1608Metric" (id 2) (at 92.456 91.186 90)
@@
   (symbol (lib_id "power:GND") (at 135.89 121.92 0)
     (in_bom yes) (on_board yes)
-    (property "Reference" "#PWR054" (id 0) (at 135.89 128.27 0)
+    (property "Reference" "#PWR058" (id 0) (at 135.89 128.27 0)
       (effects (font (size 1.27 1.27)) hide)
     )
@@
   (symbol (lib_id "Device:R_US") (at 135.89 91.44 0)
     (in_bom yes) (on_board yes)
-    (property "Reference" "R71" (id 0) (at 137.6172 90.2716 0)
+    (property "Reference" "R73" (id 0) (at 137.6172 90.2716 0)
       (effects (font (size 1.27 1.27)) (justify left))
     )
@@
   (symbol (lib_id "Device:R_US") (at 106.68 74.93 0)
     (in_bom yes) (on_board yes)
-    (property "Reference" "R70" (id 0) (at 108.4072 73.7616 0)
+    (property "Reference" "R72" (id 0) (at 108.4072 73.7616 0)
       (effects (font (size 1.27 1.27)) (justify left))
     )
@@
   (symbol (lib_id "Device:R_US") (at 135.89 100.33 0)
     (in_bom yes) (on_board yes)
-    (property "Reference" "R72" (id 0) (at 137.6172 99.1616 0)
-      (effects (font (size 1.27 1.27)) (justify left))
-    )
+    (property "Reference" "R74" (id 0) (at 137.6172 99.1616 0)
+      (effects (font (size 1.27 1.27)) (justify left))
+    )

Commit message: Driver test: updated schematic with new coarse tuning resistance values for all 3 current driver types
Parts:
- R65: renamed from R73; value 3.9 -> 4.7
- renumbered D36 to D28, D37 to D29, D38 to D30, D39 to D31, L10 to L8, Q22 to Q18, Q23 to Q19, R71 to R63, R72 to R64, R74 to R66
Changed lines of the file:
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@@
   (symbol (lib_id "Device:R_US") (at 92.71 90.17 270)
     (in_bom yes) (on_board yes)
-    (property "Reference" "R71" (id 0) (at 92.71 84.963 90))
+    (property "Reference" "R63" (id 0) (at 92.71 84.963 90))
     (property "Value" "1k" (id 1) (at 92.71 87.2744 90))
     (property "Footprint" "Resistor_SMD:R_0603_1608Metric" (id 2) (at 92.456 91.186 90)
@@
   (symbol (lib_id "Device:Q_NPN_BEC") (at 104.14 90.17 0)
     (in_bom yes) (on_board yes)
-    (property "Reference" "Q22" (id 0) (at 108.9914 89.0016 0)
+    (property "Reference" "Q18" (id 0) (at 108.9914 89.0016 0)
       (effects (font (size 1.27 1.27)) (justify left))
     )
@@
   (symbol (lib_id "Device:D_Small_Filled") (at 121.92 105.41 90)
     (in_bom yes) (on_board yes)
-    (property "Reference" "D38" (id 0) (at 123.698 104.2416 90)
+    (property "Reference" "D30" (id 0) (at 123.698 104.2416 90)
       (effects (font (size 1.27 1.27)) (justify right))
     )
@@
   (symbol (lib_id "Device:D_Small_Filled") (at 121.92 99.06 90)
     (in_bom yes) (on_board yes)
-    (property "Reference" "D37" (id 0) (at 123.698 97.8916 90)
+    (property "Reference" "D29" (id 0) (at 123.698 97.8916 90)
       (effects (font (size 1.27 1.27)) (justify right))
     )
@@
   (symbol (lib_id "Device:D_Small_Filled") (at 121.92 92.71 90)
     (in_bom yes) (on_board yes)
-    (property "Reference" "D36" (id 0) (at 123.698 91.5416 90)
+    (property "Reference" "D28" (id 0) (at 123.698 91.5416 90)
       (effects (font (size 1.27 1.27)) (justify right))
     )
@@
   (symbol (lib_id "power:GND") (at 135.89 121.92 0)
     (in_bom yes) (on_board yes)
-    (property "Reference" "#PWR058" (id 0) (at 135.89 128.27 0)
+    (property "Reference" "#PWR056" (id 0) (at 135.89 128.27 0)
       (effects (font (size 1.27 1.27)) hide)
     )
@@
   (symbol (lib_id "Device:Q_NPN_BEC") (at 133.35 81.28 0)
     (in_bom yes) (on_board yes)
-    (property "Reference" "Q23" (id 0) (at 138.2014 80.1116 0)
+    (property "Reference" "Q19" (id 0) (at 138.2014 80.1116 0)
       (effects (font (size 1.27 1.27)) (justify left))
     )
@@
   (symbol (lib_id "Device:R_US") (at 135.89 91.44 0)
     (in_bom yes) (on_board yes)
-    (property "Reference" "R73" (id 0) (at 137.6172 90.2716 0)
-      (effects (font (size 1.27 1.27)) (justify left))
-    )
-    (property "Value" "3.9" (id 1) (at 137.6172 92.583 0)
+    (property "Reference" "R65" (id 0) (at 137.6172 90.2716 0)
+      (effects (font (size 1.27 1.27)) (justify left))
+    )
+    (property "Value" "4.7" (id 1) (at 137.6172 92.583 0)
       (effects (font (size 1.27 1.27)) (justify left))
     )
@@
   (symbol (lib_id "Device:L") (at 135.89 109.22 0)
     (in_bom yes) (on_board yes)
-    (property "Reference" "L10" (id 0) (at 137.2362 108.0516 0)
+    (property "Reference" "L8" (id 0) (at 137.2362 108.0516 0)
       (effects (font (size 1.27 1.27)) (justify left))
     )
@@
   (symbol (lib_id "Device:R_US") (at 106.68 74.93 0)
     (in_bom yes) (on_board yes)
-    (property "Reference" "R72" (id 0) (at 108.4072 73.7616 0)
+    (property "Reference" "R64" (id 0) (at 108.4072 73.7616 0)
       (effects (font (size 1.27 1.27)) (justify left))
     )
@@
   (symbol (lib_id "Device:D_Small_Filled") (at 135.89 118.11 90)
     (in_bom yes) (on_board yes)
-    (property "Reference" "D39" (id 0) (at 137.668 116.9416 90)
+    (property "Reference" "D31" (id 0) (at 137.668 116.9416 90)
       (effects (font (size 1.27 1.27)) (justify right))
     )
@@
   (symbol (lib_id "Device:R_US") (at 135.89 100.33 0)
     (in_bom yes) (on_board yes)
-    (property "Reference" "R74" (id 0) (at 137.6172 99.1616 0)
-      (effects (font (size 1.27 1.27)) (justify left))
-    )
+    (property "Reference" "R66" (id 0) (at 137.6172 99.1616 0)
+      (effects (font (size 1.27 1.27)) (justify left))
+    )

Commit message: Driver test: dropped BPLSSW LED brightness by bumping its resistor up to 1k
Parts:
- renumbered D28 to D36, D29 to D37, D30 to D38, D31 to D39, L8 to L10, Q18 to Q22, Q19 to Q23, R63 to R71, R64 to R72, R65 to R73, R66 to R74
Changed lines of the file:
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@@
   (symbol (lib_id "Device:R_US") (at 92.71 90.17 270)
     (in_bom yes) (on_board yes)
-    (property "Reference" "R63" (id 0) (at 92.71 84.963 90))
+    (property "Reference" "R71" (id 0) (at 92.71 84.963 90))
     (property "Value" "1k" (id 1) (at 92.71 87.2744 90))
     (property "Footprint" "Resistor_SMD:R_0603_1608Metric" (id 2) (at 92.456 91.186 90)
@@
   (symbol (lib_id "Device:Q_NPN_BEC") (at 104.14 90.17 0)
     (in_bom yes) (on_board yes)
-    (property "Reference" "Q18" (id 0) (at 108.9914 89.0016 0)
+    (property "Reference" "Q22" (id 0) (at 108.9914 89.0016 0)
       (effects (font (size 1.27 1.27)) (justify left))
     )
@@
   (symbol (lib_id "Device:D_Small_Filled") (at 121.92 105.41 90)
     (in_bom yes) (on_board yes)
-    (property "Reference" "D30" (id 0) (at 123.698 104.2416 90)
+    (property "Reference" "D38" (id 0) (at 123.698 104.2416 90)
       (effects (font (size 1.27 1.27)) (justify right))
     )
@@
   (symbol (lib_id "Device:D_Small_Filled") (at 121.92 99.06 90)
     (in_bom yes) (on_board yes)
-    (property "Reference" "D29" (id 0) (at 123.698 97.8916 90)
+    (property "Reference" "D37" (id 0) (at 123.698 97.8916 90)
       (effects (font (size 1.27 1.27)) (justify right))
     )
@@
   (symbol (lib_id "Device:D_Small_Filled") (at 121.92 92.71 90)
     (in_bom yes) (on_board yes)
-    (property "Reference" "D28" (id 0) (at 123.698 91.5416 90)
+    (property "Reference" "D36" (id 0) (at 123.698 91.5416 90)
       (effects (font (size 1.27 1.27)) (justify right))
     )
@@
   (symbol (lib_id "power:GND") (at 135.89 121.92 0)
     (in_bom yes) (on_board yes)
-    (property "Reference" "#PWR056" (id 0) (at 135.89 128.27 0)
+    (property "Reference" "#PWR058" (id 0) (at 135.89 128.27 0)
       (effects (font (size 1.27 1.27)) hide)
     )
@@
   (symbol (lib_id "Device:Q_NPN_BEC") (at 133.35 81.28 0)
     (in_bom yes) (on_board yes)
-    (property "Reference" "Q19" (id 0) (at 138.2014 80.1116 0)
+    (property "Reference" "Q23" (id 0) (at 138.2014 80.1116 0)
       (effects (font (size 1.27 1.27)) (justify left))
     )
@@
   (symbol (lib_id "Device:R_US") (at 135.89 91.44 0)
     (in_bom yes) (on_board yes)
-    (property "Reference" "R65" (id 0) (at 137.6172 90.2716 0)
+    (property "Reference" "R73" (id 0) (at 137.6172 90.2716 0)
       (effects (font (size 1.27 1.27)) (justify left))
     )
@@
   (symbol (lib_id "Device:L") (at 135.89 109.22 0)
     (in_bom yes) (on_board yes)
-    (property "Reference" "L8" (id 0) (at 137.2362 108.0516 0)
+    (property "Reference" "L10" (id 0) (at 137.2362 108.0516 0)
       (effects (font (size 1.27 1.27)) (justify left))
     )
@@
   (symbol (lib_id "Device:R_US") (at 106.68 74.93 0)
     (in_bom yes) (on_board yes)
-    (property "Reference" "R64" (id 0) (at 108.4072 73.7616 0)
+    (property "Reference" "R72" (id 0) (at 108.4072 73.7616 0)
       (effects (font (size 1.27 1.27)) (justify left))
     )
@@
   (symbol (lib_id "Device:D_Small_Filled") (at 135.89 118.11 90)
     (in_bom yes) (on_board yes)
-    (property "Reference" "D31" (id 0) (at 137.668 116.9416 90)
+    (property "Reference" "D39" (id 0) (at 137.668 116.9416 90)
       (effects (font (size 1.27 1.27)) (justify right))
     )
@@
   (symbol (lib_id "Device:R_US") (at 135.89 100.33 0)
     (in_bom yes) (on_board yes)
-    (property "Reference" "R66" (id 0) (at 137.6172 99.1616 0)
-      (effects (font (size 1.27 1.27)) (justify left))
-    )
+    (property "Reference" "R74" (id 0) (at 137.6172 99.1616 0)
+      (effects (font (size 1.27 1.27)) (justify left))
+    )
