File: boards/driver_test/set_reset.kicad_sch (KiCad schematic)
At the start: 22 parts, among them Q5 MMBT2222, Q6 MMBT2907, Q7 MMBT2222, Q8 MMBT2222

Commit message: Driver: some high-level board rearrangement and addition of 3d models
Connections:
- net 0V renamed 4036nA
- net PWR renamed BPLIZ
Changed lines of the file:
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@@
     (stroke (width 0) (type default) (color 0 0 0 0))
   )
-  (hierarchical_label "PWR" (shape input) (at 100.33 63.5 180)
+  (hierarchical_label "BPLIZ" (shape input) (at 100.33 63.5 180)
     (effects (font (size 1.27 1.27)) (justify right))
   )
@@
     (effects (font (size 1.27 1.27)) (justify left))
   )
-  (hierarchical_label "0V" (shape input) (at 83.82 100.33 180)
+  (hierarchical_label "4036nA" (shape input) (at 83.82 100.33 180)
     (effects (font (size 1.27 1.27)) (justify right))
   )
@@
   (symbol (lib_id "power:GND") (at 128.27 132.08 0)
     (in_bom yes) (on_board yes)
-    (property "Reference" "#PWR042" (id 0) (at 128.27 138.43 0)
-      (effects (font (size 1.27 1.27)) hide)
-    )
+    (property "Reference" "#PWR045" (id 0) (at 128.27 138.43 0)
+      (effects (font (size 1.27 1.27)) hide)
+    )

Commit message: Driver test: finished up board layout
Parts:
- renumbered R33 to R35, R34 to R36, R35 to R37, R36 to R38, R37 to R39, R38 to R40, R39 to R41, R40 to R42, R41 to R43
Changed lines of the file:
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@@
   (symbol (lib_id "Device:R_US") (at 101.6 90.17 270)
     (in_bom yes) (on_board yes)
-    (property "Reference" "R33" (id 0) (at 101.6 84.963 90))
+    (property "Reference" "R35" (id 0) (at 101.6 84.963 90))
     (property "Value" "1k" (id 1) (at 101.6 87.2744 90))
     (property "Footprint" "Resistor_SMD:R_0603_1608Metric" (id 2) (at 101.346 91.186 90)
@@
   (symbol (lib_id "Device:R_US") (at 121.92 83.82 270)
     (in_bom yes) (on_board yes)
-    (property "Reference" "R34" (id 0) (at 121.92 78.613 90))
+    (property "Reference" "R36" (id 0) (at 121.92 78.613 90))
     (property "Value" "1k" (id 1) (at 121.92 80.9244 90))
     (property "Footprint" "Resistor_SMD:R_0603_1608Metric" (id 2) (at 121.666 84.836 90)
@@
   (symbol (lib_id "Device:R_US") (at 127 73.66 0)
     (in_bom yes) (on_board yes)
-    (property "Reference" "R35" (id 0) (at 128.7272 72.4916 0)
+    (property "Reference" "R37" (id 0) (at 128.7272 72.4916 0)
       (effects (font (size 1.27 1.27)) (justify left))
     )
@@
   (symbol (lib_id "Device:R_US") (at 149.86 72.39 0)
     (in_bom yes) (on_board yes)
-    (property "Reference" "R37" (id 0) (at 151.5872 71.2216 0)
+    (property "Reference" "R39" (id 0) (at 151.5872 71.2216 0)
       (effects (font (size 1.27 1.27)) (justify left))
     )
@@
   (symbol (lib_id "Device:R_US") (at 128.27 105.41 0)
     (in_bom yes) (on_board yes)
-    (property "Reference" "R36" (id 0) (at 129.9972 104.2416 0)
+    (property "Reference" "R38" (id 0) (at 129.9972 104.2416 0)
       (effects (font (size 1.27 1.27)) (justify left))
     )
@@
   (symbol (lib_id "power:GND") (at 128.27 132.08 0)
     (in_bom yes) (on_board yes)
-    (property "Reference" "#PWR045" (id 0) (at 128.27 138.43 0)
+    (property "Reference" "#PWR049" (id 0) (at 128.27 138.43 0)
       (effects (font (size 1.27 1.27)) hide)
     )
@@
   (symbol (lib_id "Device:R_US") (at 168.91 107.95 0)
     (in_bom yes) (on_board yes)
-    (property "Reference" "R38" (id 0) (at 170.6372 106.7816 0)
+    (property "Reference" "R40" (id 0) (at 170.6372 106.7816 0)
       (effects (font (size 1.27 1.27)) (justify left))
     )
@@
   (symbol (lib_id "Device:R_US") (at 185.42 104.14 0)
     (in_bom yes) (on_board yes)
-    (property "Reference" "R40" (id 0) (at 187.1472 102.9716 0)
+    (property "Reference" "R42" (id 0) (at 187.1472 102.9716 0)
       (effects (font (size 1.27 1.27)) (justify left))
     )
@@
   (symbol (lib_id "Device:R_US") (at 168.91 116.84 0)
     (in_bom yes) (on_board yes)
-    (property "Reference" "R39" (id 0) (at 170.6372 115.6716 0)
+    (property "Reference" "R41" (id 0) (at 170.6372 115.6716 0)
       (effects (font (size 1.27 1.27)) (justify left))
     )
@@
   (symbol (lib_id "Device:R_US") (at 185.42 113.03 0)
     (in_bom yes) (on_board yes)
-    (property "Reference" "R41" (id 0) (at 187.1472 111.8616 0)
-      (effects (font (size 1.27 1.27)) (justify left))
-    )
+    (property "Reference" "R43" (id 0) (at 187.1472 111.8616 0)
+      (effects (font (size 1.27 1.27)) (justify left))
+    )

Commit message: Driver test: updated schematic with new coarse tuning resistance values for all 3 current driver types
Parts:
- R51: renamed from R42; value 7.5 -> 9.1
- renumbered D9 to D16, D10 to D17, D11 to D18, D12 to D19, D13 to D20, D14 to D21, D15 to D22, L1 to L4, L2 to L5, Q6 to Q10, Q7 to Q11, Q8 to Q12, Q5 to Q9, R35 to R44, R36 to R45, R37 to R46, R38 to R47, R39 to R48, R40 to R49, R41 to R50, R43 to R52
Changed lines of the file:
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@@
   (symbol (lib_id "Device:R_US") (at 101.6 90.17 270)
     (in_bom yes) (on_board yes)
-    (property "Reference" "R35" (id 0) (at 101.6 84.963 90))
+    (property "Reference" "R44" (id 0) (at 101.6 84.963 90))
     (property "Value" "1k" (id 1) (at 101.6 87.2744 90))
     (property "Footprint" "Resistor_SMD:R_0603_1608Metric" (id 2) (at 101.346 91.186 90)
@@
   (symbol (lib_id "Device:Q_NPN_BEC") (at 113.03 90.17 0)
     (in_bom yes) (on_board yes)
-    (property "Reference" "Q5" (id 0) (at 117.8814 89.0016 0)
+    (property "Reference" "Q9" (id 0) (at 117.8814 89.0016 0)
       (effects (font (size 1.27 1.27)) (justify left))
     )
@@
   (symbol (lib_id "Device:R_US") (at 121.92 83.82 270)
     (in_bom yes) (on_board yes)
-    (property "Reference" "R36" (id 0) (at 121.92 78.613 90))
+    (property "Reference" "R45" (id 0) (at 121.92 78.613 90))
     (property "Value" "1k" (id 1) (at 121.92 80.9244 90))
     (property "Footprint" "Resistor_SMD:R_0603_1608Metric" (id 2) (at 121.666 84.836 90)
@@
   (symbol (lib_id "Device:R_US") (at 127 73.66 0)
     (in_bom yes) (on_board yes)
-    (property "Reference" "R37" (id 0) (at 128.7272 72.4916 0)
+    (property "Reference" "R46" (id 0) (at 128.7272 72.4916 0)
       (effects (font (size 1.27 1.27)) (justify left))
     )
@@
   (symbol (lib_id "Device:D_Small_Filled") (at 135.89 80.01 90)
     (in_bom yes) (on_board yes)
-    (property "Reference" "D11" (id 0) (at 137.668 78.8416 90)
+    (property "Reference" "D18" (id 0) (at 137.668 78.8416 90)
       (effects (font (size 1.27 1.27)) (justify right))
     )
@@
   (symbol (lib_id "Device:D_Small_Filled") (at 135.89 73.66 90)
     (in_bom yes) (on_board yes)
-    (property "Reference" "D10" (id 0) (at 137.668 72.4916 90)
+    (property "Reference" "D17" (id 0) (at 137.668 72.4916 90)
       (effects (font (size 1.27 1.27)) (justify right))
     )
@@
   (symbol (lib_id "Device:D_Small_Filled") (at 135.89 67.31 90)
     (in_bom yes) (on_board yes)
-    (property "Reference" "D9" (id 0) (at 137.668 66.1416 90)
+    (property "Reference" "D16" (id 0) (at 137.668 66.1416 90)
       (effects (font (size 1.27 1.27)) (justify right))
     )
@@
   (symbol (lib_id "Device:Q_PNP_BEC") (at 147.32 83.82 0) (mirror x)
     (in_bom yes) (on_board yes)
-    (property "Reference" "Q6" (id 0) (at 152.1714 82.6516 0)
+    (property "Reference" "Q10" (id 0) (at 152.1714 82.6516 0)
       (effects (font (size 1.27 1.27)) (justify left))
     )
@@
   (symbol (lib_id "Device:R_US") (at 149.86 72.39 0)
     (in_bom yes) (on_board yes)
-    (property "Reference" "R39" (id 0) (at 151.5872 71.2216 0)
+    (property "Reference" "R48" (id 0) (at 151.5872 71.2216 0)
       (effects (font (size 1.27 1.27)) (justify left))
     )
@@
   (symbol (lib_id "Device:D_Small_Filled") (at 151.13 114.3 90)
     (in_bom yes) (on_board yes)
-    (property "Reference" "D14" (id 0) (at 152.908 113.1316 90)
+    (property "Reference" "D21" (id 0) (at 152.908 113.1316 90)
       (effects (font (size 1.27 1.27)) (justify right))
     )
@@
   (symbol (lib_id "Device:D_Small_Filled") (at 151.13 107.95 90)
     (in_bom yes) (on_board yes)
-    (property "Reference" "D13" (id 0) (at 152.908 106.7816 90)
+    (property "Reference" "D20" (id 0) (at 152.908 106.7816 90)
       (effects (font (size 1.27 1.27)) (justify right))
     )
@@
   (symbol (lib_id "Device:D_Small_Filled") (at 151.13 101.6 90)
     (in_bom yes) (on_board yes)
-    (property "Reference" "D12" (id 0) (at 152.908 100.4316 90)
+    (property "Reference" "D19" (id 0) (at 152.908 100.4316 90)
       (effects (font (size 1.27 1.27)) (justify right))
     )
@@
   (symbol (lib_id "Device:D_Small_Filled") (at 151.13 120.65 90)
     (in_bom yes) (on_board yes)
-    (property "Reference" "D15" (id 0) (at 152.908 119.4816 90)
+    (property "Reference" "D22" (id 0) (at 152.908 119.4816 90)
       (effects (font (size 1.27 1.27)) (justify right))
     )
@@
   (symbol (lib_id "Device:R_US") (at 128.27 105.41 0)
     (in_bom yes) (on_board yes)
-    (property "Reference" "R38" (id 0) (at 129.9972 104.2416 0)
+    (property "Reference" "R47" (id 0) (at 129.9972 104.2416 0)
       (effects (font (size 1.27 1.27)) (justify left))
     )
@@
   (symbol (lib_id "power:GND") (at 128.27 132.08 0)
     (in_bom yes) (on_board yes)
-    (property "Reference" "#PWR046" (id 0) (at 128.27 138.43 0)
+    (property "Reference" "#PWR049" (id 0) (at 128.27 138.43 0)
       (effects (font (size 1.27 1.27)) hide)
     )
@@
   (symbol (lib_id "Device:Q_NPN_BEC") (at 166.37 97.79 0)
     (in_bom yes) (on_board yes)
-    (property "Reference" "Q7" (id 0) (at 171.2214 96.6216 0)
+    (property "Reference" "Q11" (id 0) (at 171.2214 96.6216 0)
       (effects (font (size 1.27 1.27)) (justify left))
     )
@@
   (symbol (lib_id "Device:Q_NPN_BEC") (at 182.88 90.17 0)
     (in_bom yes) (on_board yes)
-    (property "Reference" "Q8" (id 0) (at 187.7314 89.0016 0)
+    (property "Reference" "Q12" (id 0) (at 187.7314 89.0016 0)
       (effects (font (size 1.27 1.27)) (justify left))
     )
@@
   (symbol (lib_id "Device:R_US") (at 168.91 107.95 0)
     (in_bom yes) (on_board yes)
-    (property "Reference" "R40" (id 0) (at 170.6372 106.7816 0)
+    (property "Reference" "R49" (id 0) (at 170.6372 106.7816 0)
       (effects (font (size 1.27 1.27)) (justify left))
     )
@@
   (symbol (lib_id "Device:L") (at 168.91 125.73 0)
     (in_bom yes) (on_board yes)
-    (property "Reference" "L1" (id 0) (at 170.2562 124.5616 0)
+    (property "Reference" "L4" (id 0) (at 170.2562 124.5616 0)
       (effects (font (size 1.27 1.27)) (justify left))
     )
@@
   (symbol (lib_id "Device:R_US") (at 185.42 104.14 0)
     (in_bom yes) (on_board yes)
-    (property "Reference" "R42" (id 0) (at 187.1472 102.9716 0)
-      (effects (font (size 1.27 1.27)) (justify left))
-    )
-    (property "Value" "7.5" (id 1) (at 187.1472 105.283 0)
+    (property "Reference" "R51" (id 0) (at 187.1472 102.9716 0)
+      (effects (font (size 1.27 1.27)) (justify left))
+    )
+    (property "Value" "9.1" (id 1) (at 187.1472 105.283 0)
       (effects (font (size 1.27 1.27)) (justify left))
     )
@@
   (symbol (lib_id "Device:L") (at 185.42 121.92 0)
     (in_bom yes) (on_board yes)
-    (property "Reference" "L2" (id 0) (at 186.7662 120.7516 0)
+    (property "Reference" "L5" (id 0) (at 186.7662 120.7516 0)
       (effects (font (size 1.27 1.27)) (justify left))
     )
@@
   (symbol (lib_id "Device:R_US") (at 168.91 116.84 0)
     (in_bom yes) (on_board yes)
-    (property "Reference" "R41" (id 0) (at 170.6372 115.6716 0)
+    (property "Reference" "R50" (id 0) (at 170.6372 115.6716 0)
       (effects (font (size 1.27 1.27)) (justify left))
     )
@@
   (symbol (lib_id "Device:R_US") (at 185.42 113.03 0)
     (in_bom yes) (on_board yes)
-    (property "Reference" "R43" (id 0) (at 187.1472 111.8616 0)
-      (effects (font (size 1.27 1.27)) (justify left))
-    )
+    (property "Reference" "R52" (id 0) (at 187.1472 111.8616 0)
+      (effects (font (size 1.27 1.27)) (justify left))
+    )

Commit message: Driver test: dropped BPLSSW LED brightness by bumping its resistor up to 1k
Parts:
- renumbered D17 to D10, D18 to D11, D19 to D12, D20 to D13, D21 to D14, D22 to D15, D16 to D9, L4 to L1, L5 to L2, Q9 to Q5, Q10 to Q6, Q11 to Q7, Q12 to Q8, R44 to R35, R45 to R36, R46 to R37, R47 to R38, R48 to R39, R49 to R40, R50 to R41, R51 to R42, R52 to R43
Changed lines of the file:
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@@
   (symbol (lib_id "Device:R_US") (at 101.6 90.17 270)
     (in_bom yes) (on_board yes)
-    (property "Reference" "R44" (id 0) (at 101.6 84.963 90))
+    (property "Reference" "R35" (id 0) (at 101.6 84.963 90))
     (property "Value" "1k" (id 1) (at 101.6 87.2744 90))
     (property "Footprint" "Resistor_SMD:R_0603_1608Metric" (id 2) (at 101.346 91.186 90)
@@
   (symbol (lib_id "Device:Q_NPN_BEC") (at 113.03 90.17 0)
     (in_bom yes) (on_board yes)
-    (property "Reference" "Q9" (id 0) (at 117.8814 89.0016 0)
+    (property "Reference" "Q5" (id 0) (at 117.8814 89.0016 0)
       (effects (font (size 1.27 1.27)) (justify left))
     )
@@
   (symbol (lib_id "Device:R_US") (at 121.92 83.82 270)
     (in_bom yes) (on_board yes)
-    (property "Reference" "R45" (id 0) (at 121.92 78.613 90))
+    (property "Reference" "R36" (id 0) (at 121.92 78.613 90))
     (property "Value" "1k" (id 1) (at 121.92 80.9244 90))
     (property "Footprint" "Resistor_SMD:R_0603_1608Metric" (id 2) (at 121.666 84.836 90)
@@
   (symbol (lib_id "Device:R_US") (at 127 73.66 0)
     (in_bom yes) (on_board yes)
-    (property "Reference" "R46" (id 0) (at 128.7272 72.4916 0)
+    (property "Reference" "R37" (id 0) (at 128.7272 72.4916 0)
       (effects (font (size 1.27 1.27)) (justify left))
     )
@@
   (symbol (lib_id "Device:D_Small_Filled") (at 135.89 80.01 90)
     (in_bom yes) (on_board yes)
-    (property "Reference" "D18" (id 0) (at 137.668 78.8416 90)
+    (property "Reference" "D11" (id 0) (at 137.668 78.8416 90)
       (effects (font (size 1.27 1.27)) (justify right))
     )
@@
   (symbol (lib_id "Device:D_Small_Filled") (at 135.89 73.66 90)
     (in_bom yes) (on_board yes)
-    (property "Reference" "D17" (id 0) (at 137.668 72.4916 90)
+    (property "Reference" "D10" (id 0) (at 137.668 72.4916 90)
       (effects (font (size 1.27 1.27)) (justify right))
     )
@@
   (symbol (lib_id "Device:D_Small_Filled") (at 135.89 67.31 90)
     (in_bom yes) (on_board yes)
-    (property "Reference" "D16" (id 0) (at 137.668 66.1416 90)
+    (property "Reference" "D9" (id 0) (at 137.668 66.1416 90)
       (effects (font (size 1.27 1.27)) (justify right))
     )
@@
   (symbol (lib_id "Device:Q_PNP_BEC") (at 147.32 83.82 0) (mirror x)
     (in_bom yes) (on_board yes)
-    (property "Reference" "Q10" (id 0) (at 152.1714 82.6516 0)
+    (property "Reference" "Q6" (id 0) (at 152.1714 82.6516 0)
       (effects (font (size 1.27 1.27)) (justify left))
     )
@@
   (symbol (lib_id "Device:R_US") (at 149.86 72.39 0)
     (in_bom yes) (on_board yes)
-    (property "Reference" "R48" (id 0) (at 151.5872 71.2216 0)
+    (property "Reference" "R39" (id 0) (at 151.5872 71.2216 0)
       (effects (font (size 1.27 1.27)) (justify left))
     )
@@
   (symbol (lib_id "Device:D_Small_Filled") (at 151.13 114.3 90)
     (in_bom yes) (on_board yes)
-    (property "Reference" "D21" (id 0) (at 152.908 113.1316 90)
+    (property "Reference" "D14" (id 0) (at 152.908 113.1316 90)
       (effects (font (size 1.27 1.27)) (justify right))
     )
@@
   (symbol (lib_id "Device:D_Small_Filled") (at 151.13 107.95 90)
     (in_bom yes) (on_board yes)
-    (property "Reference" "D20" (id 0) (at 152.908 106.7816 90)
+    (property "Reference" "D13" (id 0) (at 152.908 106.7816 90)
       (effects (font (size 1.27 1.27)) (justify right))
     )
@@
   (symbol (lib_id "Device:D_Small_Filled") (at 151.13 101.6 90)
     (in_bom yes) (on_board yes)
-    (property "Reference" "D19" (id 0) (at 152.908 100.4316 90)
+    (property "Reference" "D12" (id 0) (at 152.908 100.4316 90)
       (effects (font (size 1.27 1.27)) (justify right))
     )
@@
   (symbol (lib_id "Device:D_Small_Filled") (at 151.13 120.65 90)
     (in_bom yes) (on_board yes)
-    (property "Reference" "D22" (id 0) (at 152.908 119.4816 90)
+    (property "Reference" "D15" (id 0) (at 152.908 119.4816 90)
       (effects (font (size 1.27 1.27)) (justify right))
     )
@@
   (symbol (lib_id "Device:R_US") (at 128.27 105.41 0)
     (in_bom yes) (on_board yes)
-    (property "Reference" "R47" (id 0) (at 129.9972 104.2416 0)
+    (property "Reference" "R38" (id 0) (at 129.9972 104.2416 0)
       (effects (font (size 1.27 1.27)) (justify left))
     )
@@
   (symbol (lib_id "power:GND") (at 128.27 132.08 0)
     (in_bom yes) (on_board yes)
-    (property "Reference" "#PWR049" (id 0) (at 128.27 138.43 0)
+    (property "Reference" "#PWR046" (id 0) (at 128.27 138.43 0)
       (effects (font (size 1.27 1.27)) hide)
     )
@@
   (symbol (lib_id "Device:Q_NPN_BEC") (at 166.37 97.79 0)
     (in_bom yes) (on_board yes)
-    (property "Reference" "Q11" (id 0) (at 171.2214 96.6216 0)
+    (property "Reference" "Q7" (id 0) (at 171.2214 96.6216 0)
       (effects (font (size 1.27 1.27)) (justify left))
     )
@@
   (symbol (lib_id "Device:Q_NPN_BEC") (at 182.88 90.17 0)
     (in_bom yes) (on_board yes)
-    (property "Reference" "Q12" (id 0) (at 187.7314 89.0016 0)
+    (property "Reference" "Q8" (id 0) (at 187.7314 89.0016 0)
       (effects (font (size 1.27 1.27)) (justify left))
     )
@@
   (symbol (lib_id "Device:R_US") (at 168.91 107.95 0)
     (in_bom yes) (on_board yes)
-    (property "Reference" "R49" (id 0) (at 170.6372 106.7816 0)
+    (property "Reference" "R40" (id 0) (at 170.6372 106.7816 0)
       (effects (font (size 1.27 1.27)) (justify left))
     )
@@
   (symbol (lib_id "Device:L") (at 168.91 125.73 0)
     (in_bom yes) (on_board yes)
-    (property "Reference" "L4" (id 0) (at 170.2562 124.5616 0)
+    (property "Reference" "L1" (id 0) (at 170.2562 124.5616 0)
       (effects (font (size 1.27 1.27)) (justify left))
     )
@@
   (symbol (lib_id "Device:R_US") (at 185.42 104.14 0)
     (in_bom yes) (on_board yes)
-    (property "Reference" "R51" (id 0) (at 187.1472 102.9716 0)
+    (property "Reference" "R42" (id 0) (at 187.1472 102.9716 0)
       (effects (font (size 1.27 1.27)) (justify left))
     )
@@
   (symbol (lib_id "Device:L") (at 185.42 121.92 0)
     (in_bom yes) (on_board yes)
-    (property "Reference" "L5" (id 0) (at 186.7662 120.7516 0)
+    (property "Reference" "L2" (id 0) (at 186.7662 120.7516 0)
       (effects (font (size 1.27 1.27)) (justify left))
     )
@@
   (symbol (lib_id "Device:R_US") (at 168.91 116.84 0)
     (in_bom yes) (on_board yes)
-    (property "Reference" "R50" (id 0) (at 170.6372 115.6716 0)
+    (property "Reference" "R41" (id 0) (at 170.6372 115.6716 0)
       (effects (font (size 1.27 1.27)) (justify left))
     )
@@
   (symbol (lib_id "Device:R_US") (at 185.42 113.03 0)
     (in_bom yes) (on_board yes)
-    (property "Reference" "R52" (id 0) (at 187.1472 111.8616 0)
-      (effects (font (size 1.27 1.27)) (justify left))
-    )
+    (property "Reference" "R43" (id 0) (at 187.1472 111.8616 0)
+      (effects (font (size 1.27 1.27)) (justify left))
+    )
