File: boards/backplane_blk2/backplane_blk2.kicad_pcb (KiCad board)
At the start: 4 copper layers, 97 x 46.2 mm, 10 parts, among them J1 Conn_04x24, J2 DIN41612_03x32_C

Commit message: Backplane: fleshed out silkscreen and finalized first revision
Other:
- board text added: "1"
- board text added: "10"
- board text added: "105"
- board text added: "110"
- board text added: "115"
- board text added: "120"
- board text added: "124"
- board text added: "15"
- board text added: "20"
- board text added: "25"
- board text added: "30"
- board text added: "32"
- board text added: "405"
- board text added: "410"
- board text added: "415"
- board text added: "420"
- board text added: "5"
- board text added: "A"
- board text added: "B"
- board text added: "Block II Backplane"
- board text added: "C"
- board text added: "Mike Stewart 2022"
Changed lines of the file:
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@@
       (effects (font (size 1 1) (thickness 0.15)))
     )
-    (fp_text user "101" (at 39.6875 4.7625) (layer "B.SilkS")
+    (fp_text user "101" (at 36.5125 6.6675) (layer "B.SilkS")
       (effects (font (size 1 1) (thickness 0.15)) (justify mirror))
     )
-    (fp_text user "401" (at 39.6875 -4.7625 180) (layer "B.SilkS")
+    (fp_text user "401" (at 36.5125 -6.6675 180) (layer "B.SilkS")
       (effects (font (size 1 1) (thickness 0.15)) (justify mirror))
     )
-    (fp_text user "424" (at -39.6875 -4.7625) (layer "B.SilkS")
+    (fp_text user "424" (at -36.5125 -6.6675) (layer "B.SilkS")
       (effects (font (size 1 1) (thickness 0.15)) (justify mirror))
     )
-    (fp_text user "124" (at -39.6875 4.7625) (layer "B.SilkS")
+    (fp_text user "J1" (at -39.6875 4.7625) (layer "B.SilkS") hide
       (effects (font (size 1 1) (thickness 0.15)) (justify mirror))
     )
-    (fp_text user "101" (at 39.6875 4.7625) (layer "F.SilkS")
+    (fp_text user "101" (at 36.5125 6.6675) (layer "F.SilkS")
       (effects (font (size 1 1) (thickness 0.15)))
     )
-    (fp_text user "424" (at -39.6875 -4.7625) (layer "F.SilkS")
+    (fp_text user "424" (at -36.5125 -6.6675) (layer "F.SilkS")
       (effects (font (size 1 1) (thickness 0.15)))
     )
-    (fp_text user "124" (at -39.6875 4.7625) (layer "F.SilkS")
+    (fp_text user "124" (at -36.5125 6.6675) (layer "F.SilkS")
       (effects (font (size 1 1) (thickness 0.15)))
     )
-    (fp_text user "401" (at 39.6875 -4.7625) (layer "F.SilkS")
+    (fp_text user "401" (at 36.5125 -6.6675) (layer "F.SilkS")
       (effects (font (size 1 1) (thickness 0.15)))
     )
@@
   (gr_line (start 202.184 74.3585) (end 202.184 120.5865) (layer "Edge.Cuts") (width 0.05))
   (gr_line (start 105.156 74.3585) (end 202.184 74.3585) (layer "Edge.Cuts") (width 0.05))
+  (gr_text "120" (at 129.8575 115.57) (layer "B.SilkS")
+    (effects (font (size 1 1) (thickness 0.15)) (justify mirror))
+  )
+  (gr_text "25" (at 175.26 82.042) (layer "B.SilkS")
+    (effects (font (size 1 1) (thickness 0.15)) (justify mirror))
+  )
+  (gr_text "32" (at 193.04 82.042) (layer "B.SilkS")
+    (effects (font (size 1 1) (thickness 0.15)) (justify mirror))
+  )
+  (gr_text "Mike Stewart 2022" (at 120.142 119.126) (layer "B.SilkS")
+    (effects (font (size 1 1) (thickness 0.15)) (justify mirror))
+  )
+  (gr_text "124" (at 117.1575 115.57) (layer "B.SilkS")
+    (effects (font (size 1 1) (thickness 0.15)) (justify mirror))
+  )
+  (gr_text "B" (at 112.776 86.36) (layer "B.SilkS")
+    (effects (font (size 1 1) (thickness 0.15)) (justify mirror))
+  )
+  (gr_text "420" (at 129.8575 102.235) (layer "B.SilkS")
+    (effects (font (size 1 1) (thickness 0.15)) (justify mirror))
+  )
+  (gr_text "5" (at 124.46 82.042) (layer "B.SilkS")
+    (effects (font (size 1 1) (thickness 0.15)) (justify mirror))
+  )
+  (gr_text "110" (at 161.6075 115.57) (layer "B.SilkS")
+    (effects (font (size 1 1) (thickness 0.15)) (justify mirror))
+  )
+  (gr_text "105" (at 177.4825 115.57) (layer "B.SilkS")
+    (effects (font (size 1 1) (thickness 0.15)) (justify mirror))
+  )
+  (gr_text "115" (at 145.7325 115.57) (layer "B.SilkS")
+    (effects (font (size 1 1) (thickness 0.15)) (justify mirror))
+  )
+  (gr_text "415" (at 146.3675 102.235) (layer "B.SilkS")
+    (effects (font (size 1 1) (thickness 0.15)) (justify mirror))
+  )
+  (gr_text "15" (at 149.86 82.042) (layer "B.SilkS")
+    (effects (font (size 1 1) (thickness 0.15)) (justify mirror))
+  )
+  (gr_text "C" (at 112.776 83.82) (layer "B.SilkS")
+    (effects (font (size 1 1) (thickness 0.15)) (justify mirror))
+  )
+  (gr_text "405" (at 177.4825 102.235) (layer "B.SilkS")
+    (effects (font (size 1 1) (thickness 0.15)) (justify mirror))
+  )
+  (gr_text "A" (at 112.776 88.9) (layer "B.SilkS")
+    (effects (font (size 1 1) (thickness 0.15)) (justify mirror))
+  )
+  (gr_text "Block II Backplane" (at 186.944 119.126) (layer "B.SilkS")
+    (effects (font (size 1 1) (thickness 0.15)) (justify mirror))
+  )
+  (gr_text "30" (at 187.96 82.042) (layer "B.SilkS")
+    (effects (font (size 1 1) (thickness 0.15)) (justify mirror))
+  )
+  (gr_text "20" (at 162.56 82.042) (layer "B.SilkS")
+    (effects (font (size 1 1) (thickness 0.15)) (justify mirror))
+  )
+  (gr_text "1" (at 114.3 82.042) (layer "B.SilkS")
+    (effects (font (size 1 1) (thickness 0.15)) (justify mirror))
+  )
+  (gr_text "10" (at 137.16 82.042) (layer "B.SilkS")
+    (effects (font (size 1 1) (thickness 0.15)) (justify mirror))
+  )
+  (gr_text "410" (at 161.6075 102.235) (layer "B.SilkS")
+    (effects (font (size 1 1) (thickness 0.15)) (justify mirror))
+  )
   (segment (start 114.3 101.2825) (end 114.3 88.9) (width 0.254) (layer "B.Cu") (net 1))
   (segment (start 117.1575 104.14) (end 114.3 101.2825) (width 0.254) (layer "B.Cu") (net 1))
